File: overhead/lights/electronics/lights.kicad_sch (KiCad schematic)
At the start: 84 parts, among them J1 Conn_02x01, J2 Conn_02x13_Counter_Clockwise, J3 Conn_02x01, J4 Conn_02x01, J5 Conn_02x01, J6 Conn_02x01

Commit message: Light Panel Schematic
Parts:
- removed J2: Conn_02x13_Counter_Clockwise, Connector_PinHeader_2.54mm:PinHeader_2x14_P2.54mm_Vertical, symbol Connector_Generic:Conn_02x14_Counter_Clockwise
- removed J3, J4, J5, J6: Conn_02x01, Connector_PinHeader_2.54mm:PinHeader_1x02_P2.54mm_Vertical, symbol Connector_Generic:Conn_02x01
- added J10, J11, J18, J19, J20, J21, J8, J9: Conn_01x03_Pin, Connector_PinHeader_2.54mm:PinHeader_1x03_P2.54mm_Vertical, symbol Connector:Conn_01x03_Pin
- added J12, J13, J14, J15, J2, J22, J23, J24, J25: Conn_01x04_Pin, symbol Connector:Conn_01x04_Pin
- added J17: Conn_01x09_Pin, symbol Connector:Conn_01x09_Pin
- added J3: Conn_02x37_Counter_Clockwise, Connector_PinHeader_2.54mm:PinHeader_2x37_P2.54mm_Vertical, symbol Connector_Generic:Conn_02x37_Counter_Clockwise
- added KR9: ~, OpenA3XX:Korry Switch, symbol KorrySwitch:Korry_Switch
Connections:
- net GND: now also KR1.1 (+5V_TOP_LED), KR1.3 (+5V_BOTTOM_LED), KR1.5 (SW_IN), KR7.2 (GND_TOP_LED), KR7.4 (GND_BOTTOM_LED), KR7.6 (SW_OUT), KR8.2 (GND_TOP_LED), KR8.4 (GND_BOTTOM_LED), KR8.6 (SW_OUT), J10.1 (Pin_1), J11.1 (Pin_1), J12.1 (Pin_1), J13.1 (Pin_1), J14.1 (Pin_1), J15.1 (Pin_1), J17.1 (Pin_1), J2.1 (Pin_1), J20.1 (Pin_1), J21.1 (Pin_1), J22.1 (Pin_1), J23.1 (Pin_1), J24.1 (Pin_1), J25.1 (Pin_1), J3.1 (Pin_1), J3.2 (Pin_2), J3.3 (Pin_3), J8.1 (Pin_1), J9.1 (Pin_1), KR9.2 (GND_TOP_LED), KR9.4 (GND_BOTTOM_LED), KR9.6 (SW_OUT)
- net at KR4.1 (+5V_TOP_LED): now also J3.19 (Pin_19)
- net at KR4.3 (+5V_BOTTOM_LED): now also J3.20 (Pin_20)
- net at KR4.5 (SW_IN): now also J3.21 (Pin_21)
- net at KR2.1 (+5V_TOP_LED): now also J3.16 (Pin_16)
- net at KR2.3 (+5V_BOTTOM_LED): now also J3.17 (Pin_17)
- net at KR2.5 (SW_IN): now also J3.18 (Pin_18)
- net at KR6.1 (+5V_TOP_LED): now also J3.22 (Pin_22)
- net at KR6.3 (+5V_BOTTOM_LED): now also J3.23 (Pin_23)
- net at KR6.5 (SW_IN): now also J3.25 (Pin_25)
- net at KR7.1 (+5V_TOP_LED): now also J3.10 (Pin_10)
- net at KR7.3 (+5V_BOTTOM_LED): now also J3.11 (Pin_11)
- net at KR7.5 (SW_IN): now also J3.12 (Pin_12)
- net at KR8.1 (+5V_TOP_LED): now also J3.24 (Pin_24)
- net at KR8.3 (+5V_BOTTOM_LED): now also J3.26 (Pin_26)
- net at KR8.5 (SW_IN): now also J3.27 (Pin_27)
- net at KR3.1 (+5V_TOP_LED): now also J3.4 (Pin_4)
- net at KR3.3 (+5V_BOTTOM_LED): now also J3.5 (Pin_5)
- net at KR3.5 (SW_IN): now also J3.6 (Pin_6)
- net at KR5.1 (+5V_TOP_LED): now also J3.7 (Pin_7)
- net at KR5.3 (+5V_BOTTOM_LED): now also J3.8 (Pin_8)
- net at KR5.5 (SW_IN): now also J3.9 (Pin_9)
- new net: J18.3 (Pin_3), J19.1 (Pin_1)
- new net: J18.2 (Pin_2), J19.2 (Pin_2)
- new net: J18.1 (Pin_1), J19.3 (Pin_3)
- new net: J3.13 (Pin_13), KR9.1 (+5V_TOP_LED)
- new net: J3.14 (Pin_14), KR9.3 (+5V_BOTTOM_LED)
- new net: J3.15 (Pin_15), KR9.5 (SW_IN)
Other:
- note removed: "Flap Mode"
- note removed: "G/S Mode"
- note removed: "GEN 1 Line"
- note removed: "GND CTL"
- note removed: "LDG Flap 3"
- note removed: "RAT & EMER GEN"
- note removed: "SYS"
- note removed: "TERR"
- moved on the sheet: J1, KR4

Commit message: Lights Panel Continuation
Parts:
- removed J3: Conn_02x37_Counter_Clockwise, Connector_PinHeader_2.54mm:PinHeader_2x37_P2.54mm_Vertical, symbol Connector_Generic:Conn_02x37_Counter_Clockwise
- added J1, J10: Conn_02x20_Counter_Clockwise, Connector_PinHeader_2.54mm:PinHeader_2x20_P2.54mm_Vertical, symbol Connector_Generic:Conn_02x20_Counter_Clockwise
- J12: renamed from J2; footprint (none) -> Connector_PinHeader_2.54mm:PinHeader_1x04_P2.54mm_Vertical
- J13: renamed from J17; footprint (none) -> Connector_PinHeader_2.54mm:PinHeader_1x09_P2.54mm_Vertical
- J16: renamed from J22; footprint (none) -> Connector_PinHeader_2.54mm:PinHeader_1x04_P2.54mm_Vertical
- J17: renamed from J23; footprint (none) -> Connector_PinHeader_2.54mm:PinHeader_1x04_P2.54mm_Vertical
- J18: renamed from J24; footprint (none) -> Connector_PinHeader_2.54mm:PinHeader_1x04_P2.54mm_Vertical
- J19: renamed from J25; footprint (none) -> Connector_PinHeader_2.54mm:PinHeader_1x04_P2.54mm_Vertical
- J20: renamed from J19; footprint Connector_PinHeader_2.54mm:PinHeader_1x03_P2.54mm_Vertical -> TerminalBlock:TerminalBlock_bornier-3_P5.08mm
- J6: renamed from J12; footprint (none) -> Connector_PinHeader_2.54mm:PinHeader_1x04_P2.54mm_Vertical
- J7: renamed from J13; footprint (none) -> Connector_PinHeader_2.54mm:PinHeader_1x04_P2.54mm_Vertical
- J8: renamed from J14; footprint (none) -> Connector_PinHeader_2.54mm:PinHeader_1x04_P2.54mm_Vertical
- J9: renamed from J15; footprint (none) -> Connector_PinHeader_2.54mm:PinHeader_1x04_P2.54mm_Vertical
- renumbered J18 to J11, J20 to J14, J21 to J15, J8 to J2, J1 to J21, J9 to J3, J11 to J4, J10 to J5
Connections:
- net GND: no longer KR1.1 (+5V_TOP_LED), KR1.3 (+5V_BOTTOM_LED), KR1.5 (SW_IN)
- net at J12.2 (Pin_2): now also J10.10 (Pin_10)
- net at J12.3 (Pin_3): now also J10.11 (Pin_11)
- net at J12.4 (Pin_4): now also J10.12 (Pin_12)
- net at J15.2 (Pin_2): now also J10.23 (Pin_23)
- net at J15.3 (Pin_3): now also J10.24 (Pin_24)
- net at J5.2 (Pin_2): now also J1.34 (Pin_34)
- net at J5.3 (Pin_3): now also J1.35 (Pin_35)
- net at J6.2 (Pin_2): now also J1.36 (Pin_36)
- net at J6.3 (Pin_3): now also J1.37 (Pin_37)
- net at J6.4 (Pin_4): now also J1.38 (Pin_38)
- net at KR4.1 (+5V_TOP_LED): now also J1.19 (Pin_19)
- net at KR4.3 (+5V_BOTTOM_LED): now also J1.20 (Pin_20)
- net at KR4.5 (SW_IN): now also J1.21 (Pin_21)
- net at J2.2 (Pin_2): now also J1.29 (Pin_29)
- net at J2.3 (Pin_3): now also J1.28 (Pin_28)
- net at J14.2 (Pin_2): now also J10.21 (Pin_21)
- net at J14.3 (Pin_3): now also J10.22 (Pin_22)
- net at J7.2 (Pin_2): now also J10.1 (Pin_1)
- net at J7.3 (Pin_3): now also J10.2 (Pin_2)
- net at J7.4 (Pin_4): now also J10.3 (Pin_3)
- net at J9.2 (Pin_2): now also J10.7 (Pin_7)
- net at J9.3 (Pin_3): now also J10.8 (Pin_8)
- net at J9.4 (Pin_4): now also J10.9 (Pin_9)
- net at KR7.1 (+5V_TOP_LED): now also J1.10 (Pin_10)
- net at KR7.3 (+5V_BOTTOM_LED): now also J1.11 (Pin_11)
- net at KR7.5 (SW_IN): now also J1.12 (Pin_12)
- net at KR9.1 (+5V_TOP_LED): now also J1.13 (Pin_13)
- net at KR9.3 (+5V_BOTTOM_LED): now also J1.14 (Pin_14)
- net at KR9.5 (SW_IN): now also J1.15 (Pin_15)
- net at KR2.1 (+5V_TOP_LED): now also J1.16 (Pin_16)
- net at KR2.3 (+5V_BOTTOM_LED): now also J1.17 (Pin_17)
- net at KR2.5 (SW_IN): now also J1.18 (Pin_18)
- net at KR6.1 (+5V_TOP_LED): now also J1.22 (Pin_22)
- net at KR6.3 (+5V_BOTTOM_LED): now also J1.23 (Pin_23)
- net at KR8.1 (+5V_TOP_LED): now also J1.24 (Pin_24)
- net at KR6.5 (SW_IN): now also J1.25 (Pin_25)
- net at KR8.3 (+5V_BOTTOM_LED): now also J1.26 (Pin_26)
- net at KR8.5 (SW_IN): now also J1.27 (Pin_27)
- net at KR3.1 (+5V_TOP_LED): now also J1.4 (Pin_4)
- net at KR3.3 (+5V_BOTTOM_LED): now also J1.5 (Pin_5)
- net at KR3.5 (SW_IN): now also J1.6 (Pin_6)
- net at KR5.1 (+5V_TOP_LED): now also J1.7 (Pin_7)
- net at KR5.3 (+5V_BOTTOM_LED): now also J1.8 (Pin_8)
- net at KR5.5 (SW_IN): now also J1.9 (Pin_9)
- net at J16.2 (Pin_2): now also J10.25 (Pin_25)
- net at J16.3 (Pin_3): now also J10.26 (Pin_26)
- net at J16.4 (Pin_4): now also J10.27 (Pin_27)
- net at J3.2 (Pin_2): now also J1.30 (Pin_30)
- net at J3.3 (Pin_3): now also J1.31 (Pin_31)
- net at J18.2 (Pin_2): now also J10.31 (Pin_31)
- net at J18.3 (Pin_3): now also J10.32 (Pin_32)
- net at J18.4 (Pin_4): now also J10.33 (Pin_33)
- net at J19.2 (Pin_2): now also J10.34 (Pin_34)
- net at J19.3 (Pin_3): now also J10.35 (Pin_35)
- net at J19.4 (Pin_4): now also J10.36 (Pin_36)
- net at J4.2 (Pin_2): now also J1.32 (Pin_32)
- net at J4.3 (Pin_3): now also J1.33 (Pin_33)
- net at J17.2 (Pin_2): now also J10.28 (Pin_28)
- net at J17.3 (Pin_3): now also J10.29 (Pin_29)
- net at J17.4 (Pin_4): now also J10.30 (Pin_30)
- net at J8.2 (Pin_2): now also J10.4 (Pin_4)
- net at J8.3 (Pin_3): now also J10.5 (Pin_5)
- net at J8.4 (Pin_4): now also J10.6 (Pin_6)
- net at J13.2 (Pin_2): now also J10.13 (Pin_13)
- net at J13.3 (Pin_3): now also J10.14 (Pin_14)
- net at J13.4 (Pin_4): now also J10.15 (Pin_15)
- net at J13.5 (Pin_5): now also J10.16 (Pin_16)
- net at J13.6 (Pin_6): now also J10.17 (Pin_17)
- net at J13.7 (Pin_7): now also J10.18 (Pin_18)
- net at J13.8 (Pin_8): now also J10.19 (Pin_19)
- net at J13.9 (Pin_9): now also J10.20 (Pin_20)
- new net: J1.1 (Pin_1), KR1.1 (+5V_TOP_LED)
- new net: J1.2 (Pin_2), KR1.3 (+5V_BOTTOM_LED)
- new net: J1.3 (Pin_3), KR1.5 (SW_IN)
Other:
- moved on the sheet: J11, J12, J13, J14, J15, J16, J17, J18, J19, J20, J21

Commit message: Light Panels - Progress
Parts:
- added D100, D101, D102, D103, D104, D105, D106, D107, D108, D109, D110, D111, D112, D113, D114, D115, D116, D53, D54, D55, D56, D57, D58, D59, D60, D61, D62, D63, D64, D65, D66, D67, D68, D69, D70, D71, D72, D73, D74, D75, D76, D77, D78, D79, D80, D81, D82, D83, D84, D85, D86, D87, D88, D89, D90, D91, D92, D93, D94, D95, D96, D97, D98, D99: LED, OpenA3XX:LED_Everlight-SMD3528_3.5x2.8mm_67-21ST, symbol Device:LED
- added R19, R20, R21, R22, R23, R24, R25, R26, R27, R28, R29, R30, R31, R32, R33, R34, R35, R36, R37, R38, R39, R40: 220R, Resistor_SMD:R_1206_3216Metric_Pad1.30x1.75mm_HandSolder, symbol Device:R
Connections:
- net +12V: now also D102.2 (A), D105.2 (A), D108.2 (A), D111.2 (A), D114.2 (A), D53.2 (A), D56.2 (A), D59.2 (A), D62.2 (A), D65.2 (A), D68.2 (A), D71.2 (A), D74.2 (A), D75.2 (A), D78.2 (A), D81.2 (A), D84.2 (A), D87.2 (A), D90.2 (A), D93.2 (A), D96.2 (A), D99.2 (A)
- net GND: now also R19.2, R20.2, R21.2, R22.2, R23.2, R24.2, R25.2, R26.2, R27.2, R28.2, R29.2, R30.2, R31.2, R32.2, R33.2, R34.2, R35.2, R36.2, R37.2, R38.2, R39.2, R40.2
- new net: D86.1 (K), R30.1
- new net: D109.1 (K), D110.2 (A)
- new net: D108.1 (K), D109.2 (A)
- new net: D54.1 (K), D55.2 (A)
- new net: D53.1 (K), D54.2 (A)
- new net: D101.1 (K), R35.1
- new net: D65.1 (K), D66.2 (A)
- new net: D80.1 (K), R28.1
- new net: D74.1 (K), R26.1
- new net: D89.1 (K), R31.1
- new net: D88.1 (K), D89.2 (A)
- new net: D102.1 (K), D103.2 (A)
- new net: D90.1 (K), D91.2 (A)
- new net: D75.1 (K), D76.2 (A)
- new net: D55.1 (K), R19.1
- new net: D76.1 (K), D77.2 (A)
- new net: D112.1 (K), D113.2 (A)
- new net: D111.1 (K), D112.2 (A)
- new net: D105.1 (K), D106.2 (A)
- new net: D95.1 (K), R33.1
- new net: D91.1 (K), D92.2 (A)
- new net: D59.1 (K), D60.2 (A)
- new net: D61.1 (K), R21.1
- new net: D87.1 (K), D88.2 (A)
- new net: D85.1 (K), D86.2 (A)
- new net: D84.1 (K), D85.2 (A)
- new net: D73.1 (K), R25.1
- new net: D68.1 (K), D69.2 (A)
- new net: D77.1 (K), R27.1
- new net: D113.1 (K), R39.1
- new net: D79.1 (K), D80.2 (A)
- new net: D78.1 (K), D79.2 (A)
- new net: D100.1 (K), D101.2 (A)
- new net: D70.1 (K), R24.1
- new net: D69.1 (K), D70.2 (A)
- new net: D98.1 (K), R34.1
- new net: D64.1 (K), R22.1
- new net: D63.1 (K), D64.2 (A)
- new net: D104.1 (K), R36.1
- new net: D56.1 (K), D57.2 (A)
- new net: D115.1 (K), D116.2 (A)
- new net: D114.1 (K), D115.2 (A)
- new net: D60.1 (K), D61.2 (A)
- new net: D83.1 (K), R29.1
- new net: D82.1 (K), D83.2 (A)
- new net: D92.1 (K), R32.1
- new net: D97.1 (K), D98.2 (A)
- new net: D96.1 (K), D97.2 (A)
- new net: D107.1 (K), R37.1
- new net: D106.1 (K), D107.2 (A)
- new net: D72.1 (K), D73.2 (A)
- new net: D71.1 (K), D72.2 (A)
- new net: D116.1 (K), R40.1
- new net: D93.1 (K), D94.2 (A)
- new net: D67.1 (K), R23.1
- new net: D103.1 (K), D104.2 (A)
- new net: D58.1 (K), R20.1
- new net: D57.1 (K), D58.2 (A)
- new net: D66.1 (K), D67.2 (A)
- new net: D94.1 (K), D95.2 (A)
- new net: D62.1 (K), D63.2 (A)
- new net: D81.1 (K), D82.2 (A)
- new net: D100.2 (A), D99.1 (K)
- new net: D110.1 (K), R38.1
