File: overhead/aircond/electronics/aircond/aircond.kicad_pcb (KiCad board)
At the start: 2 copper layers, 0 parts

Commit message: Aircond Panel!
Parts:
- added D1: LED, OpenA3XX:LED_Everlight-SMD3528_3.5x2.8mm_67-21ST, F.Cu at (59.6, 111.8)
- added D10: LED, OpenA3XX:LED_Everlight-SMD3528_3.5x2.8mm_67-21ST, F.Cu at (79.8, 127.8)
- added D100: LED, OpenA3XX:LED_Everlight-SMD3528_3.5x2.8mm_67-21ST, F.Cu at (340.0, 97.2)
- added D101: LED, OpenA3XX:LED_Everlight-SMD3528_3.5x2.8mm_67-21ST, F.Cu at (312.6, 96.3)
- added D102: LED, OpenA3XX:LED_Everlight-SMD3528_3.5x2.8mm_67-21ST, F.Cu at (310.6, 114.7)
- added D103: LED, OpenA3XX:LED_Everlight-SMD3528_3.5x2.8mm_67-21ST, F.Cu at (267.7, 128.7)
- added D104: LED, OpenA3XX:LED_Everlight-SMD3528_3.5x2.8mm_67-21ST, F.Cu at (256.2, 128.3)
- added D105: LED, OpenA3XX:LED_Everlight-SMD3528_3.5x2.8mm_67-21ST, F.Cu at (280.5, 116.5)
- added D106: LED, OpenA3XX:LED_Everlight-SMD3528_3.5x2.8mm_67-21ST, F.Cu at (367.5, 112.9)
- added D107: LED, OpenA3XX:LED_Everlight-SMD3528_3.5x2.8mm_67-21ST, F.Cu at (278.3, 104.2)
- added D108: LED, OpenA3XX:LED_Everlight-SMD3528_3.5x2.8mm_67-21ST, F.Cu at (272.3, 96.0)
- added D109: LED, OpenA3XX:LED_Everlight-SMD3528_3.5x2.8mm_67-21ST, F.Cu at (255.1, 96.2)
- added D11: LED, OpenA3XX:LED_Everlight-SMD3528_3.5x2.8mm_67-21ST, F.Cu at (93.5, 133.2)
- added D110: LED, OpenA3XX:LED_Everlight-SMD3528_3.5x2.8mm_67-21ST, F.Cu at (244.5, 106.2)
- added D111: LED, OpenA3XX:LED_Everlight-SMD3528_3.5x2.8mm_67-21ST, F.Cu at (245.7, 118.0)
- added D112: LED, OpenA3XX:LED_Everlight-SMD3528_3.5x2.8mm_67-21ST, F.Cu at (229.2, 136.8)
- added D113: LED, OpenA3XX:LED_Everlight-SMD3528_3.5x2.8mm_67-21ST, F.Cu at (230.2, 118.8)
- added D114: LED, OpenA3XX:LED_Everlight-SMD3528_3.5x2.8mm_67-21ST, F.Cu at (229.6, 105.0)
- added D115: LED, OpenA3XX:LED_Everlight-SMD3528_3.5x2.8mm_67-21ST, F.Cu at (245.4, 89.3)
- added D116: LED, OpenA3XX:LED_Everlight-SMD3528_3.5x2.8mm_67-21ST, F.Cu at (222.0, 96.2)
- added D117: LED, OpenA3XX:LED_Everlight-SMD3528_3.5x2.8mm_67-21ST, F.Cu at (204.8, 96.3)
- added D118: LED, OpenA3XX:LED_Everlight-SMD3528_3.5x2.8mm_67-21ST, F.Cu at (229.1, 89.5)
- added D119: LED, OpenA3XX:LED_Everlight-SMD3528_3.5x2.8mm_67-21ST, F.Cu at (196.3, 89.5)
- added D12: LED, OpenA3XX:LED_Everlight-SMD3528_3.5x2.8mm_67-21ST, F.Cu at (72.5, 164.1)
- added D120: LED, OpenA3XX:LED_Everlight-SMD3528_3.5x2.8mm_67-21ST, F.Cu at (196.7, 104.2)
- added D121: LED, OpenA3XX:LED_Everlight-SMD3528_3.5x2.8mm_67-21ST, F.Cu at (196.3, 117.5)
- added D122: LED, OpenA3XX:LED_Everlight-SMD3528_3.5x2.8mm_67-21ST, F.Cu at (217.2, 128.8)
- added D13: LED, OpenA3XX:LED_Everlight-SMD3528_3.5x2.8mm_67-21ST, F.Cu at (89.8, 164.5)
- added D14: LED, OpenA3XX:LED_Everlight-SMD3528_3.5x2.8mm_67-21ST, F.Cu at (106.4, 134.1)
- added D15: LED, OpenA3XX:LED_Everlight-SMD3528_3.5x2.8mm_67-21ST, F.Cu at (106.7, 148.8)
- added D16: LED, OpenA3XX:LED_Everlight-SMD3528_3.5x2.8mm_67-21ST, F.Cu at (120.4, 157.6)
- added D17: LED, OpenA3XX:LED_Everlight-SMD3528_3.5x2.8mm_67-21ST, F.Cu at (97.0, 151.1)
- added D18: LED, OpenA3XX:LED_Everlight-SMD3528_3.5x2.8mm_67-21ST, F.Cu at (99.0, 164.5)
- added D19: LED, OpenA3XX:LED_Everlight-SMD3528_3.5x2.8mm_67-21ST, F.Cu at (98.5, 177.5)
- added D2: LED, OpenA3XX:LED_Everlight-SMD3528_3.5x2.8mm_67-21ST, F.Cu at (81.8, 104.5)
- added D20: LED, OpenA3XX:LED_Everlight-SMD3528_3.5x2.8mm_67-21ST, F.Cu at (61.0, 190.4)
- added D21: LED, OpenA3XX:LED_Everlight-SMD3528_3.5x2.8mm_67-21ST, F.Cu at (77.6, 188.1)
- added D22: LED, OpenA3XX:LED_Everlight-SMD3528_3.5x2.8mm_67-21ST, F.Cu at (99.0, 190.6)
- added D23: LED, OpenA3XX:LED_Everlight-SMD3528_3.5x2.8mm_67-21ST, F.Cu at (114.2, 186.3)
- added D24: LED, OpenA3XX:LED_Everlight-SMD3528_3.5x2.8mm_67-21ST, F.Cu at (129.0, 190.5)
- added D25: LED, OpenA3XX:LED_Everlight-SMD3528_3.5x2.8mm_67-21ST, F.Cu at (129.5, 176.6)
- added D26: LED, OpenA3XX:LED_Everlight-SMD3528_3.5x2.8mm_67-21ST, F.Cu at (131.5, 151.6)
- added D27: LED, OpenA3XX:LED_Everlight-SMD3528_3.5x2.8mm_67-21ST, F.Cu at (122.2, 128.8)
- added D28: LED, OpenA3XX:LED_Everlight-SMD3528_3.5x2.8mm_67-21ST, F.Cu at (130.4, 141.4)
- added D29: LED, OpenA3XX:LED_Everlight-SMD3528_3.5x2.8mm_67-21ST, F.Cu at (139.2, 128.9)
- added D3: LED, OpenA3XX:LED_Everlight-SMD3528_3.5x2.8mm_67-21ST, F.Cu at (92.8, 94.8)
- added D30: LED, OpenA3XX:LED_Everlight-SMD3528_3.5x2.8mm_67-21ST, F.Cu at (151.8, 136.1)
- added D31: LED, OpenA3XX:LED_Everlight-SMD3528_3.5x2.8mm_67-21ST, F.Cu at (139.8, 161.2)
- added D32: LED, OpenA3XX:LED_Everlight-SMD3528_3.5x2.8mm_67-21ST, F.Cu at (152.2, 151.4)
- added D33: LED, OpenA3XX:LED_Everlight-SMD3528_3.5x2.8mm_67-21ST, F.Cu at (157.3, 128.4)
- added D34: LED, OpenA3XX:LED_Everlight-SMD3528_3.5x2.8mm_67-21ST, F.Cu at (145.9, 116.7)
- added D35: LED, OpenA3XX:LED_Everlight-SMD3528_3.5x2.8mm_67-21ST, F.Cu at (147.2, 103.0)
- added D36: LED, OpenA3XX:LED_Everlight-SMD3528_3.5x2.8mm_67-21ST, F.Cu at (155.0, 96.0)
- added D37: LED, OpenA3XX:LED_Everlight-SMD3528_3.5x2.8mm_67-21ST, F.Cu at (170.4, 95.9)
- added D38: LED, OpenA3XX:LED_Everlight-SMD3528_3.5x2.8mm_67-21ST, F.Cu at (147.2, 89.2)
- added D39: LED, OpenA3XX:LED_Everlight-SMD3528_3.5x2.8mm_67-21ST, F.Cu at (179.6, 89.3)
- added D4: LED, OpenA3XX:LED_Everlight-SMD3528_3.5x2.8mm_67-21ST, F.Cu at (112.1, 105.1)
- added D40: LED, OpenA3XX:LED_Everlight-SMD3528_3.5x2.8mm_67-21ST, F.Cu at (178.4, 103.4)
- added D41: LED, OpenA3XX:LED_Everlight-SMD3528_3.5x2.8mm_67-21ST, F.Cu at (180.1, 115.8)
- added D42: LED, OpenA3XX:LED_Everlight-SMD3528_3.5x2.8mm_67-21ST, F.Cu at (169.1, 128.3)
- added D43: LED, OpenA3XX:LED_Everlight-SMD3528_3.5x2.8mm_67-21ST, F.Cu at (179.8, 136.0)
- added D44: LED, OpenA3XX:LED_Everlight-SMD3528_3.5x2.8mm_67-21ST, F.Cu at (161.9, 140.9)
- added D45: LED, OpenA3XX:LED_Everlight-SMD3528_3.5x2.8mm_67-21ST, F.Cu at (173.0, 141.1)
- added D46: LED, OpenA3XX:LED_Everlight-SMD3528_3.5x2.8mm_67-21ST, F.Cu at (181.0, 150.9)
- added D47: LED, OpenA3XX:LED_Everlight-SMD3528_3.5x2.8mm_67-21ST, F.Cu at (190.1, 129.4)
- added D48: LED, OpenA3XX:LED_Everlight-SMD3528_3.5x2.8mm_67-21ST, F.Cu at (201.8, 135.9)
- added D49: LED, OpenA3XX:LED_Everlight-SMD3528_3.5x2.8mm_67-21ST, F.Cu at (202.2, 150.9)
- added D5: LED, OpenA3XX:LED_Everlight-SMD3528_3.5x2.8mm_67-21ST, F.Cu at (103.2, 94.8)
- added D50: LED, OpenA3XX:LED_Everlight-SMD3528_3.5x2.8mm_67-21ST, F.Cu at (167.3, 155.8)
- added D51: LED, OpenA3XX:LED_Everlight-SMD3528_3.5x2.8mm_67-21ST, F.Cu at (151.8, 166.6)
- added D52: LED, OpenA3XX:LED_Everlight-SMD3528_3.5x2.8mm_67-21ST, F.Cu at (151.2, 178.6)
- added D53: LED, OpenA3XX:LED_Everlight-SMD3528_3.5x2.8mm_67-21ST, F.Cu at (152.3, 190.4)
- added D54: LED, OpenA3XX:LED_Everlight-SMD3528_3.5x2.8mm_67-21ST, F.Cu at (168.1, 186.8)
- added D55: LED, OpenA3XX:LED_Everlight-SMD3528_3.5x2.8mm_67-21ST, F.Cu at (182.8, 190.7)
- added D56: LED, OpenA3XX:LED_Everlight-SMD3528_3.5x2.8mm_67-21ST, F.Cu at (182.8, 176.3)
- added D57: LED, OpenA3XX:LED_Everlight-SMD3528_3.5x2.8mm_67-21ST, F.Cu at (190.1, 168.0)
- added D58: LED, OpenA3XX:LED_Everlight-SMD3528_3.5x2.8mm_67-21ST, F.Cu at (190.4, 157.8)
- added D59: LED, OpenA3XX:LED_Everlight-SMD3528_3.5x2.8mm_67-21ST, F.Cu at (197.9, 176.7)
- added D6: LED, OpenA3XX:LED_Everlight-SMD3528_3.5x2.8mm_67-21ST, F.Cu at (62.1, 127.7)
- added D60: LED, OpenA3XX:LED_Everlight-SMD3528_3.5x2.8mm_67-21ST, F.Cu at (198.3, 190.6)
- added D61: LED, OpenA3XX:LED_Everlight-SMD3528_3.5x2.8mm_67-21ST, F.Cu at (213.3, 186.9)
- added D62: LED, OpenA3XX:LED_Everlight-SMD3528_3.5x2.8mm_67-21ST, F.Cu at (227.5, 190.2)
- added D63: LED, OpenA3XX:LED_Everlight-SMD3528_3.5x2.8mm_67-21ST, F.Cu at (228.1, 177.4)
- added D64: LED, OpenA3XX:LED_Everlight-SMD3528_3.5x2.8mm_67-21ST, F.Cu at (227.7, 162.2)
- added D65: LED, OpenA3XX:LED_Everlight-SMD3528_3.5x2.8mm_67-21ST, F.Cu at (208.9, 157.7)
- added D66: LED, OpenA3XX:LED_Everlight-SMD3528_3.5x2.8mm_67-21ST, F.Cu at (225.5, 151.2)
- added D67: LED, OpenA3XX:LED_Everlight-SMD3528_3.5x2.8mm_67-21ST, F.Cu at (249.5, 150.8)
- added D68: LED, OpenA3XX:LED_Everlight-SMD3528_3.5x2.8mm_67-21ST, F.Cu at (253.4, 159.8)
- added D69: LED, OpenA3XX:LED_Everlight-SMD3528_3.5x2.8mm_67-21ST, F.Cu at (247.4, 169.9)
- added D7: LED, OpenA3XX:LED_Everlight-SMD3528_3.5x2.8mm_67-21ST, F.Cu at (63.4, 148.8)
- added D70: LED, OpenA3XX:LED_Everlight-SMD3528_3.5x2.8mm_67-21ST, F.Cu at (271.8, 159.3)
- added D71: LED, OpenA3XX:LED_Everlight-SMD3528_3.5x2.8mm_67-21ST, F.Cu at (278.4, 169.2)
- added D72: LED, OpenA3XX:LED_Everlight-SMD3528_3.5x2.8mm_67-21ST, F.Cu at (252.1, 190.2)
- added D73: LED, OpenA3XX:LED_Everlight-SMD3528_3.5x2.8mm_67-21ST, F.Cu at (274.7, 189.9)
- added D74: LED, OpenA3XX:LED_Everlight-SMD3528_3.5x2.8mm_67-21ST, F.Cu at (287.9, 152.3)
- added D75: LED, OpenA3XX:LED_Everlight-SMD3528_3.5x2.8mm_67-21ST, F.Cu at (263.2, 147.9)
- added D76: LED, OpenA3XX:LED_Everlight-SMD3528_3.5x2.8mm_67-21ST, F.Cu at (249.3, 137.4)
- added D77: LED, OpenA3XX:LED_Everlight-SMD3528_3.5x2.8mm_67-21ST, F.Cu at (272.6, 137.2)
- added D78: LED, OpenA3XX:LED_Everlight-SMD3528_3.5x2.8mm_67-21ST, F.Cu at (304.5, 151.4)
- added D79: LED, OpenA3XX:LED_Everlight-SMD3528_3.5x2.8mm_67-21ST, F.Cu at (295.4, 164.9)
- added D8: LED, OpenA3XX:LED_Everlight-SMD3528_3.5x2.8mm_67-21ST, F.Cu at (60.1, 170.1)
- added D80: LED, OpenA3XX:LED_Everlight-SMD3528_3.5x2.8mm_67-21ST, F.Cu at (294.6, 179.3)
- added D81: LED, OpenA3XX:LED_Everlight-SMD3528_3.5x2.8mm_67-21ST, F.Cu at (295.3, 190.9)
- added D82: LED, OpenA3XX:LED_Everlight-SMD3528_3.5x2.8mm_67-21ST, F.Cu at (310.6, 186.8)
- added D83: LED, OpenA3XX:LED_Everlight-SMD3528_3.5x2.8mm_67-21ST, F.Cu at (326.2, 188.6)
- added D84: LED, OpenA3XX:LED_Everlight-SMD3528_3.5x2.8mm_67-21ST, F.Cu at (325.8, 176.7)
- added D85: LED, OpenA3XX:LED_Everlight-SMD3528_3.5x2.8mm_67-21ST, F.Cu at (353.4, 188.7)
- added D86: LED, OpenA3XX:LED_Everlight-SMD3528_3.5x2.8mm_67-21ST, F.Cu at (366.5, 170.2)
- added D87: LED, OpenA3XX:LED_Everlight-SMD3528_3.5x2.8mm_67-21ST, F.Cu at (366.8, 139.1)
- added D88: LED, OpenA3XX:LED_Everlight-SMD3528_3.5x2.8mm_67-21ST, F.Cu at (355.9, 133.1)
- added D89: LED, OpenA3XX:LED_Everlight-SMD3528_3.5x2.8mm_67-21ST, F.Cu at (359.0, 149.1)
- added D9: LED, OpenA3XX:LED_Everlight-SMD3528_3.5x2.8mm_67-21ST, F.Cu at (68.7, 133.6)
- added D90: LED, OpenA3XX:LED_Everlight-SMD3528_3.5x2.8mm_67-21ST, F.Cu at (345.0, 163.1)
- added D91: LED, OpenA3XX:LED_Everlight-SMD3528_3.5x2.8mm_67-21ST, F.Cu at (327.8, 154.6)
- added D92: LED, OpenA3XX:LED_Everlight-SMD3528_3.5x2.8mm_67-21ST, F.Cu at (328.2, 138.2)
- added D93: LED, OpenA3XX:LED_Everlight-SMD3528_3.5x2.8mm_67-21ST, F.Cu at (343.6, 128.4)
- added D94: LED, OpenA3XX:LED_Everlight-SMD3528_3.5x2.8mm_67-21ST, F.Cu at (317.6, 149.8)
- added D95: LED, OpenA3XX:LED_Everlight-SMD3528_3.5x2.8mm_67-21ST, F.Cu at (293.3, 141.6)
- added D96: LED, OpenA3XX:LED_Everlight-SMD3528_3.5x2.8mm_67-21ST, F.Cu at (314.6, 134.1)
- added D97: LED, OpenA3XX:LED_Everlight-SMD3528_3.5x2.8mm_67-21ST, F.Cu at (292.6, 128.4)
- added D98: LED, OpenA3XX:LED_Everlight-SMD3528_3.5x2.8mm_67-21ST, F.Cu at (326.4, 126.2)
- added D99: LED, OpenA3XX:LED_Everlight-SMD3528_3.5x2.8mm_67-21ST, F.Cu at (341.9, 114.0)
- added J1: Conn_02x20_Counter_Clockwise, Connector_PinHeader_2.54mm:PinHeader_2x20_P2.54mm_Vertical, B.Cu at (138.5, 89.8)
- added J2: Conn_01x09_Pin, Connector_PinHeader_2.54mm:PinHeader_1x09_P2.54mm_Vertical, F.Cu at (152.8, 112.3)
- added J3: Conn_01x09_Pin, Connector_PinHeader_2.54mm:PinHeader_1x09_P2.54mm_Vertical, F.Cu at (203.1, 112.0)
- added J4: Conn_01x09_Pin, Connector_PinHeader_2.54mm:PinHeader_1x09_P2.54mm_Vertical, F.Cu at (252.5, 112.0)
- added J5: Conn_01x04_Pin, Connector_PinHeader_2.54mm:PinHeader_1x04_P2.54mm_Vertical, F.Cu at (94.2, 113.5)
- added J6: Conn_01x04_Pin, Connector_PinHeader_2.54mm:PinHeader_1x04_P2.54mm_Vertical, F.Cu at (258.8, 178.1)
- added J7: Conn_02x20_Counter_Clockwise, Connector_PinHeader_2.54mm:PinHeader_2x20_P2.54mm_Vertical, B.Cu at (331.2, 90.1)
- added J8: Conn_02x01, TerminalBlock:TerminalBlock_bornier-2_P5.08mm, B.Cu at (68.5, 87.0)
- added KR1: ~, OpenA3XX:Korry Switch, F.Cu at (70.8, 138.2)
- added KR2: ~, OpenA3XX:Korry Switch, F.Cu at (103.8, 168.0)
- added KR3: ~, OpenA3XX:Korry Switch, F.Cu at (333.2, 138.0)
- added KR4: ~, OpenA3XX:Korry Switch, F.Cu at (157.2, 167.8)
- added KR5: ~, OpenA3XX:Korry Switch, F.Cu at (300.1, 168.1)
- added KR6: ~, OpenA3XX:Korry Switch, F.Cu at (315.9, 101.5)
- added KR7: ~, OpenA3XX:Korry Switch, F.Cu at (202.6, 167.9)
- added R1: 220R, Resistor_SMD:R_1206_3216Metric_Pad1.30x1.75mm_HandSolder, F.Cu at (82.0, 110.9)
- added R10: 220R, Resistor_SMD:R_1206_3216Metric_Pad1.30x1.75mm_HandSolder, F.Cu at (130.9, 160.9)
- added R11: 220R, Resistor_SMD:R_1206_3216Metric_Pad1.30x1.75mm_HandSolder, F.Cu at (151.6, 158.6)
- added R12: 220R, Resistor_SMD:R_1206_3216Metric_Pad1.30x1.75mm_HandSolder, F.Cu at (139.9, 141.1)
- added R13: 220R, Resistor_SMD:R_1206_3216Metric_Pad1.30x1.75mm_HandSolder, F.Cu at (179.9, 96.0)
- added R14: 220R, Resistor_SMD:R_1206_3216Metric_Pad1.30x1.75mm_HandSolder, F.Cu at (187.4, 103.5)
- added R15: 220R, Resistor_SMD:R_1206_3216Metric_Pad1.30x1.75mm_HandSolder, F.Cu at (187.8, 119.8)
- added R16: 220R, Resistor_SMD:R_1206_3216Metric_Pad1.30x1.75mm_HandSolder, F.Cu at (190.4, 143.6)
- added R17: 220R, Resistor_SMD:R_1206_3216Metric_Pad1.30x1.75mm_HandSolder, F.Cu at (209.3, 143.2)
- added R18: 220R, Resistor_SMD:R_1206_3216Metric_Pad1.30x1.75mm_HandSolder, F.Cu at (140.0, 176.9)
- added R19: 220R, Resistor_SMD:R_1206_3216Metric_Pad1.30x1.75mm_HandSolder, F.Cu at (190.7, 183.8)
- added R2: 220R, Resistor_SMD:R_1206_3216Metric_Pad1.30x1.75mm_HandSolder, F.Cu at (79.7, 122.0)
- added R20: 220R, Resistor_SMD:R_1206_3216Metric_Pad1.30x1.75mm_HandSolder, F.Cu at (190.4, 136.8)
- added R21: 220R, Resistor_SMD:R_1206_3216Metric_Pad1.30x1.75mm_HandSolder, F.Cu at (238.4, 184.1)
- added R22: 220R, Resistor_SMD:R_1206_3216Metric_Pad1.30x1.75mm_HandSolder, F.Cu at (237.6, 171.5)
- added R23: 220R, Resistor_SMD:R_1206_3216Metric_Pad1.30x1.75mm_HandSolder, F.Cu at (237.2, 143.4)
- added R24: 220R, Resistor_SMD:R_1206_3216Metric_Pad1.30x1.75mm_HandSolder, F.Cu at (273.8, 151.1)
- added R25: 220R, Resistor_SMD:R_1206_3216Metric_Pad1.30x1.75mm_HandSolder, F.Cu at (280.2, 182.7)
- added R26: 220R, Resistor_SMD:R_1206_3216Metric_Pad1.30x1.75mm_HandSolder, F.Cu at (288.1, 172.7)
- added R27: 220R, Resistor_SMD:R_1206_3216Metric_Pad1.30x1.75mm_HandSolder, F.Cu at (283.4, 141.3)
- added R28: 220R, Resistor_SMD:R_1206_3216Metric_Pad1.30x1.75mm_HandSolder, F.Cu at (286.4, 189.3)
- added R29: 220R, Resistor_SMD:R_1206_3216Metric_Pad1.30x1.75mm_HandSolder, F.Cu at (335.8, 184.2)
- added R3: 220R, Resistor_SMD:R_1206_3216Metric_Pad1.30x1.75mm_HandSolder, F.Cu at (96.8, 141.6)
- added R30: 220R, Resistor_SMD:R_1206_3216Metric_Pad1.30x1.75mm_HandSolder, F.Cu at (353.0, 180.2)
- added R31: 220R, Resistor_SMD:R_1206_3216Metric_Pad1.30x1.75mm_HandSolder, F.Cu at (352.6, 170.3)
- added R32: 220R, Resistor_SMD:R_1206_3216Metric_Pad1.30x1.75mm_HandSolder, F.Cu at (359.7, 162.8)
- added R33: 220R, Resistor_SMD:R_1206_3216Metric_Pad1.30x1.75mm_HandSolder, F.Cu at (283.7, 128.0)
- added R34: 220R, Resistor_SMD:R_1206_3216Metric_Pad1.30x1.75mm_HandSolder, F.Cu at (307.4, 126.7)
- added R35: 220R, Resistor_SMD:R_1206_3216Metric_Pad1.30x1.75mm_HandSolder, F.Cu at (305.4, 106.0)
- added R36: 220R, Resistor_SMD:R_1206_3216Metric_Pad1.30x1.75mm_HandSolder, F.Cu at (237.7, 128.9)
- added R37: 220R, Resistor_SMD:R_1206_3216Metric_Pad1.30x1.75mm_HandSolder, F.Cu at (293.2, 106.0)
- added R38: 220R, Resistor_SMD:R_1206_3216Metric_Pad1.30x1.75mm_HandSolder, F.Cu at (244.9, 98.5)
- added R39: 220R, Resistor_SMD:R_1206_3216Metric_Pad1.30x1.75mm_HandSolder, F.Cu at (237.4, 112.0)
- added R4: 220R, Resistor_SMD:R_1206_3216Metric_Pad1.30x1.75mm_HandSolder, F.Cu at (65.0, 159.7)
- added R40: 220R, Resistor_SMD:R_1206_3216Metric_Pad1.30x1.75mm_HandSolder, F.Cu at (234.4, 96.6)
- added R41: 220R, Resistor_SMD:R_1206_3216Metric_Pad1.30x1.75mm_HandSolder, F.Cu at (191.2, 96.0)
- added R42: 220R, Resistor_SMD:R_1206_3216Metric_Pad1.30x1.75mm_HandSolder, F.Cu at (219.2, 136.6)
- added R5: 220R, Resistor_SMD:R_1206_3216Metric_Pad1.30x1.75mm_HandSolder, F.Cu at (106.2, 156.2)
- added R6: 220R, Resistor_SMD:R_1206_3216Metric_Pad1.30x1.75mm_HandSolder, F.Cu at (89.8, 172.7)
- added R7: 220R, Resistor_SMD:R_1206_3216Metric_Pad1.30x1.75mm_HandSolder, F.Cu at (88.5, 186.7)
- added R8: 220R, Resistor_SMD:R_1206_3216Metric_Pad1.30x1.75mm_HandSolder, F.Cu at (140.2, 184.1)
- added R9: 220R, Resistor_SMD:R_1206_3216Metric_Pad1.30x1.75mm_HandSolder, F.Cu at (139.7, 169.4)
- added bottom: LOGO, OpenA3XX:OpenA3XXLogoSmall, B.Cu at (72.0, 110.5)
- added top: LOGO, OpenA3XX:OpenA3XXLogoSmall, F.Cu at (71.8, 110.5)
Routing:
- net GND: track 0.00 -> 1346.0 mm, vias 0 -> 19
- net +12V: track 0.00 -> 1200.0 mm, vias 0 -> 27
- net Net-(J1-Pin_5): track 0.00 -> 276.3 mm, vias 0 -> 2
- net Net-(J1-Pin_7): track 0.00 -> 274.8 mm, vias 0 -> 2
- net Net-(J1-Pin_4): track 0.00 -> 274.3 mm, vias 0 -> 3
- net Net-(J1-Pin_8): track 0.00 -> 271.6 mm, vias 0 -> 1
- net Net-(J1-Pin_6): track 0.00 -> 267.0 mm, vias 0 -> 2
- net Net-(J5-Pin_2): track 0.00 -> 261.9 mm, vias 0 -> 1
- net Net-(J5-Pin_1): track 0.00 -> 256.1 mm, vias 0 -> 1
- net Net-(J1-Pin_9): track 0.00 -> 251.0 mm, vias 0 -> 1
- net Net-(J5-Pin_3): track 0.00 -> 248.6 mm, vias 0 -> 2
- net Net-(J1-Pin_11): track 0.00 -> 227.7 mm, vias 0 -> 2
- net Net-(J1-Pin_12): track 0.00 -> 221.3 mm, vias 0 -> 2
- net Net-(J1-Pin_10): track 0.00 -> 219.2 mm, vias 0 -> 1
- net Net-(J1-Pin_14): track 0.00 -> 179.8 mm, vias 0 -> 1
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Other:
- board outline added: 322.4 x 112.7 mm
- board text added: "Flight Simulation Only"
- board text added: "KR5"
- board text added: "https://www.github.com/OpenA3XX - AIR COND V1.0"
- board text added: "~"
- board text added: "© 2025 OpenA3XX • CC BY-SA 4.0"
