File: overhead/aircond/electronics/aircond/aircond.kicad_sch (KiCad schematic)
At the start: 0 parts

Commit message: Aircond Panel!
Parts:
- added D1, D10, D100, D101, D102, D103, D104, D105, D106, D107, D108, D109, D11, D110, D111, D112, D113, D114, D115, D116, D117, D118, D119, D12, D120, D121, D122, D13, D14, D15, D16, D17, D18, D19, D2, D20, D21, D22, D23, D24, D25, D26, D27, D28, D29, D3, D30, D31, D32, D33, D34, D35, D36, D37, D38, D39, D4, D40, D41, D42, D43, D44, D45, D46, D47, D48, D49, D5, D50, D51, D52, D53, D54, D55, D56, D57, D58, D59, D6, D60, D61, D62, D63, D64, D65, D66, D67, D68, D69, D7, D70, D71, D72, D73, D74, D75, D76, D77, D78, D79, D8, D80, D81, D82, D83, D84, D85, D86, D87, D88, D89, D9, D90, D91, D92, D93, D94, D95, D96, D97, D98, D99: LED, OpenA3XX:LED_Everlight-SMD3528_3.5x2.8mm_67-21ST, symbol Device:LED
- added J1, J7: Conn_02x20_Counter_Clockwise, Connector_PinHeader_2.54mm:PinHeader_2x20_P2.54mm_Vertical, symbol Connector_Generic:Conn_02x20_Counter_Clockwise
- added J2, J3, J4: Conn_01x09_Pin, Connector_PinHeader_2.54mm:PinHeader_1x09_P2.54mm_Vertical, symbol Connector:Conn_01x09_Pin
- added J5, J6: Conn_01x04_Pin, Connector_PinHeader_2.54mm:PinHeader_1x04_P2.54mm_Vertical, symbol Connector:Conn_01x04_Pin
- added J8: Conn_02x01, TerminalBlock:TerminalBlock_bornier-2_P5.08mm, symbol Connector_Generic:Conn_02x01
- added KR1, KR2, KR3, KR4, KR5, KR6, KR7: ~, OpenA3XX:Korry Switch, symbol KorrySwitch:Korry_Switch
- added R1, R10, R11, R12, R13, R14, R15, R16, R17, R18, R19, R2, R20, R21, R22, R23, R24, R25, R26, R27, R28, R29, R3, R30, R31, R32, R33, R34, R35, R36, R37, R38, R39, R4, R40, R41, R42, R5, R6, R7, R8, R9: 220R, Resistor_SMD:R_1206_3216Metric_Pad1.30x1.75mm_HandSolder, symbol Device:R
Connections:
- new net: J6.1 (Pin_1), J7.12 (Pin_12)
- new net: J6.2 (Pin_2), J7.13 (Pin_13)
- new net: J6.3 (Pin_3), J7.14 (Pin_14)
- new net: D86.1 (K), R30.1
- new net: D31.1 (K), R11.1
- new net: D20.1 (K), D21.2 (A)
- new net: D19.1 (K), D20.2 (A)
- new net: D109.1 (K), D110.2 (A)
- new net: D108.1 (K), D109.2 (A)
- new net: D54.1 (K), D55.2 (A)
- new net: D53.1 (K), D54.2 (A)
- new net: D12.1 (K), R4.1
- new net: D101.1 (K), R35.1
- new net: D5.1 (K), D6.2 (A)
- new net: D4.1 (K), D5.2 (A)
- new net: D34.1 (K), R12.1
- new net: D33.1 (K), D34.2 (A)
- new net: D65.1 (K), D66.2 (A)
- new net: D6.1 (K), R2.1
- new net: D80.1 (K), R28.1
- new net: D74.1 (K), R26.1
- new net: D24.1 (K), D25.2 (A)
- new net: D23.1 (K), D24.2 (A)
- new net: D89.1 (K), R31.1
- new net: D88.1 (K), D89.2 (A)
- new net: D102.1 (K), D103.2 (A)
- new net: D3.1 (K), R1.1
- new net: D32.1 (K), D33.2 (A)
- new net: D90.1 (K), D91.2 (A)
- new net: D37.1 (K), R13.1
- new net: D75.1 (K), D76.2 (A)
- new net: D55.1 (K), R19.1
- new net: D30.1 (K), D31.2 (A)
- new net: D29.1 (K), D30.2 (A)
- new net: D76.1 (K), D77.2 (A)
- new net: D112.1 (K), D113.2 (A)
- new net: D111.1 (K), D112.2 (A)
- new net: J4.2 (Pin_2), J7.1 (Pin_1)
- new net: J5.2 (Pin_2), J7.10 (Pin_10)
- new net: J5.3 (Pin_3), J7.11 (Pin_11)
- new net: J4.3 (Pin_3), J7.2 (Pin_2)
- new net: J4.4 (Pin_4), J7.3 (Pin_3)
- new net: J4.5 (Pin_5), J7.4 (Pin_4)
- new net: J4.6 (Pin_6), J7.5 (Pin_5)
- new net: J4.7 (Pin_7), J7.6 (Pin_6)
- new net: J4.8 (Pin_8), J7.7 (Pin_7)
- new net: J4.9 (Pin_9), J7.8 (Pin_8)
- new net: J5.1 (Pin_1), J7.9 (Pin_9)
- new net: D105.1 (K), D106.2 (A)
- new net: J1.19 (Pin_19), KR4.1 (+5V_TOP_LED)
- new net: J1.20 (Pin_20), KR4.3 (+5V_BOTTOM_LED)
- new net: J1.21 (Pin_21), KR4.5 (SW_IN)
- new net: D117.1 (K), D118.2 (A)
- new net: D95.1 (K), R33.1
- new net: D91.1 (K), D92.2 (A)
- new net: D59.1 (K), D60.2 (A)
- new net: D22.1 (K), R8.1
- new net: D61.1 (K), R21.1
- new net: D8.1 (K), D9.2 (A)
- new net: D7.1 (K), D8.2 (A)
- new net: D87.1 (K), D88.2 (A)
- new net: D85.1 (K), D86.2 (A)
- new net: D84.1 (K), D85.2 (A)
- new net: D73.1 (K), R25.1
- new net: D46.1 (K), R16.1
- new net: D45.1 (K), D46.2 (A)
- new net: D28.1 (K), R10.1
- new net: D27.1 (K), D28.2 (A)
- new net: D68.1 (K), D69.2 (A)
- new net: D77.1 (K), R27.1
- new net: D25.1 (K), R9.1
- new net: D13.1 (K), D14.2 (A)
- new net: D122.1 (K), R42.1
- new net: D121.1 (K), D122.2 (A)
- new net: D43.1 (K), R15.1
- new net: D113.1 (K), R39.1
- new net: D49.1 (K), R17.1
- new net: D79.1 (K), D80.2 (A)
- new net: D78.1 (K), D79.2 (A)
- new net: D26.1 (K), D27.2 (A)
- new net: D100.1 (K), D101.2 (A)
- new net: D70.1 (K), R24.1
- new net: D69.1 (K), D70.2 (A)
- new net: D98.1 (K), R34.1
- new net: D119.1 (K), R41.1
- new net: D48.1 (K), D49.2 (A)
- new net: D64.1 (K), R22.1
- new net: D63.1 (K), D64.2 (A)
- new net: D47.1 (K), D48.2 (A)
- new net: D104.1 (K), R36.1
- new net: D56.1 (K), D57.2 (A)
- new net: D51.1 (K), D52.2 (A)
- new net: D50.1 (K), D51.2 (A)
- new net: D115.1 (K), D116.2 (A)
- new net: D114.1 (K), D115.2 (A)
- new net: D36.1 (K), D37.2 (A)
- new net: J1.30 (Pin_30), J3.2 (Pin_2)
- new net: J1.31 (Pin_31), J3.3 (Pin_3)
- new net: J1.32 (Pin_32), J3.4 (Pin_4)
- new net: J1.33 (Pin_33), J3.5 (Pin_5)
- new net: J1.34 (Pin_34), J3.6 (Pin_6)
- new net: J1.35 (Pin_35), J3.7 (Pin_7)
- new net: J1.36 (Pin_36), J3.8 (Pin_8)
- new net: J1.37 (Pin_37), J3.9 (Pin_9)
- new net: D52.1 (K), R18.1
- new net: D60.1 (K), D61.2 (A)
- new net: D15.1 (K), R5.1
- new net: D14.1 (K), D15.2 (A)
- new net: D41.1 (K), D42.2 (A)
- new net: D42.1 (K), D43.2 (A)
- new net: D83.1 (K), R29.1
- new net: D82.1 (K), D83.2 (A)
- new net: D9.1 (K), R3.1
- new net: D92.1 (K), R32.1
- new net: D97.1 (K), D98.2 (A)
- new net: D96.1 (K), D97.2 (A)
- new net: D107.1 (K), R37.1
- new net: D106.1 (K), D107.2 (A)
- new net: D35.1 (K), D36.2 (A)
- new net: J1.1 (Pin_1), KR1.1 (+5V_TOP_LED)
- new net: J1.10 (Pin_10), KR6.1 (+5V_TOP_LED)
- new net: J1.11 (Pin_11), KR6.3 (+5V_BOTTOM_LED)
- new net: J1.12 (Pin_12), KR6.5 (SW_IN)
- new net: J1.13 (Pin_13), KR7.1 (+5V_TOP_LED)
- new net: J1.14 (Pin_14), KR7.3 (+5V_BOTTOM_LED)
- new net: J1.15 (Pin_15), KR7.5 (SW_IN)
- new net: J1.16 (Pin_16), KR2.1 (+5V_TOP_LED)
- new net: J1.17 (Pin_17), KR2.3 (+5V_BOTTOM_LED)
- new net: J1.18 (Pin_18), KR2.5 (SW_IN)
- new net: J1.2 (Pin_2), KR1.3 (+5V_BOTTOM_LED)
- new net: J1.22 (Pin_22), J2.2 (Pin_2)
- new net: J1.23 (Pin_23), J2.3 (Pin_3)
- new net: J1.24 (Pin_24), J2.4 (Pin_4)
- new net: J1.25 (Pin_25), J2.5 (Pin_5)
- new net: J1.26 (Pin_26), J2.6 (Pin_6)
- new net: J1.27 (Pin_27), J2.7 (Pin_7)
- new net: J1.28 (Pin_28), J2.8 (Pin_8)
- new net: J1.29 (Pin_29), J2.9 (Pin_9)
- new net: J1.3 (Pin_3), KR1.5 (SW_IN)
- new net: J1.4 (Pin_4), KR3.1 (+5V_TOP_LED)
- new net: J1.5 (Pin_5), KR3.3 (+5V_BOTTOM_LED)
- new net: J1.6 (Pin_6), KR3.5 (SW_IN)
- new net: J1.7 (Pin_7), KR5.1 (+5V_TOP_LED)
- new net: J1.8 (Pin_8), KR5.3 (+5V_BOTTOM_LED)
- new net: J1.9 (Pin_9), KR5.5 (SW_IN)
- new net: D11.1 (K), D12.2 (A)
- new net: D72.1 (K), D73.2 (A)
- new net: D71.1 (K), D72.2 (A)
- new net: D118.1 (K), D119.2 (A)
- new net: D116.1 (K), R40.1
- new net: D38.1 (K), D39.2 (A)
- new net: D93.1 (K), D94.2 (A)
- new net: D18.1 (K), R6.1
- new net: D67.1 (K), R23.1
- new net: D103.1 (K), D104.2 (A)
- new net: D44.1 (K), D45.2 (A)
- new net: D1.1 (K), D2.2 (A)
- new net: D58.1 (K), R20.1
- new net: D57.1 (K), D58.2 (A)
- new net: D2.1 (K), D3.2 (A)
- new net: D120.1 (K), D121.2 (A)
- new net: D66.1 (K), D67.2 (A)
- new net: D17.1 (K), D18.2 (A)
- new net: D16.1 (K), D17.2 (A)
- new net: D10.1 (K), D11.2 (A)
- new net: D21.1 (K), R7.1
- new net: D94.1 (K), D95.2 (A)
- new net: D62.1 (K), D63.2 (A)
- new net: D81.1 (K), D82.2 (A)
- new net: D40.1 (K), R14.1
- new net: D39.1 (K), D40.2 (A)
- new net: D100.2 (A), D99.1 (K)
- new net: D110.1 (K), R38.1
- new net +12V: D1.2 (A), D10.2 (A), D102.2 (A), D105.2 (A), D108.2 (A), D111.2 (A), D114.2 (A), D117.2 (A), D120.2 (A), D13.2 (A), D16.2 (A), D19.2 (A), D22.2 (A), D23.2 (A), D26.2 (A), D29.2 (A), D32.2 (A), D35.2 (A), D38.2 (A), D4.2 (A), D41.2 (A), D44.2 (A), D47.2 (A), D50.2 (A), D53.2 (A), D56.2 (A), D59.2 (A), D62.2 (A), D65.2 (A), D68.2 (A), D7.2 (A), D71.2 (A), D74.2 (A), D75.2 (A), D78.2 (A), D81.2 (A), D84.2 (A), D87.2 (A), D90.2 (A), D93.2 (A), D96.2 (A), D99.2 (A), J8.2 (Pin_2)
- new net GND: J2.1 (Pin_1), J3.1 (Pin_1), J4.1 (Pin_1), J5.4 (Pin_4), J6.4 (Pin_4), J8.1 (Pin_1), KR1.2 (GND_TOP_LED), KR1.4 (GND_BOTTOM_LED), KR1.6 (SW_OUT), KR2.2 (GND_TOP_LED), KR2.4 (GND_BOTTOM_LED), KR2.6 (SW_OUT), KR3.2 (GND_TOP_LED), KR3.4 (GND_BOTTOM_LED), KR3.6 (SW_OUT), KR4.2 (GND_TOP_LED), KR4.4 (GND_BOTTOM_LED), KR4.6 (SW_OUT), KR5.2 (GND_TOP_LED), KR5.4 (GND_BOTTOM_LED), KR5.6 (SW_OUT), KR6.2 (GND_TOP_LED), KR6.4 (GND_BOTTOM_LED), KR6.6 (SW_OUT), KR7.2 (GND_TOP_LED), KR7.4 (GND_BOTTOM_LED), KR7.6 (SW_OUT), R1.2, R10.2, R11.2, R12.2, R13.2, R14.2, R15.2, R16.2, R17.2, R18.2, R19.2, R2.2, R20.2, R21.2, R22.2, R23.2, R24.2, R25.2, R26.2, R27.2, R28.2, R29.2, R3.2, R30.2, R31.2, R32.2, R33.2, R34.2, R35.2, R36.2, R37.2, R38.2, R39.2, R4.2, R40.2, R41.2, R42.2, R5.2, R6.2, R7.2, R8.2, R9.2
- no-connect marks 0 -> 29
