File: overhead/elec/electronics/elec.kicad_pcb (KiCad board)
At the start: 2 copper layers, 322.3 x 106.5 mm, 0 parts

Commit message: Elec PCB continuation
Parts:
- added C2: 10uF, Capacitor_THT:CP_Radial_D5.0mm_P2.50mm, B.Cu at (176.6, 146.9)
- added C3: 0.1 uF, Capacitor_SMD:C_1206_3216Metric_Pad1.33x1.80mm_HandSolder, B.Cu at (197.3, 146.8)
- added D1: 1N5818, Diode_SMD:D_SMA_Handsoldering, B.Cu at (346.8, 106.7)
- added IC1: MAX7219CWG, Package_SO:SOIC-24W_7.5x15.4mm_P1.27mm, B.Cu at (187.1, 146.7)
- added J1: Conn_02x20_Counter_Clockwise, Connector_PinHeader_2.54mm:PinHeader_2x20_P2.54mm_Vertical, B.Cu at (328.5, 100.0)
- added J21: Conn_02x01, TerminalBlock:TerminalBlock_bornier-2_P5.08mm, B.Cu at (60.3, 99.2)
- added KR1: ~, OpenA3XX:Korry Switch, F.Cu at (71.5, 106.1)
- added KR10: ~, OpenA3XX:Korry Switch, F.Cu at (328.1, 169.8)
- added KR11: ~, OpenA3XX:Korry Switch, F.Cu at (174.2, 108.2)
- added KR12: ~, OpenA3XX:Korry Switch, F.Cu at (201.2, 108.2)
- added KR2: ~, OpenA3XX:Korry Switch, F.Cu at (71.2, 136.8)
- added KR3: ~, OpenA3XX:Korry Switch, F.Cu at (71.2, 169.6)
- added KR4: ~, OpenA3XX:Korry Switch, F.Cu at (102.5, 169.9)
- added KR5: ~, OpenA3XX:Korry Switch, F.Cu at (160.7, 170.0)
- added KR6: ~, OpenA3XX:Korry Switch, F.Cu at (201.2, 152.4)
- added KR7: ~, OpenA3XX:Korry Switch, F.Cu at (242.2, 170.0)
- added KR8: ~, OpenA3XX:Korry Switch, F.Cu at (268.1, 121.2)
- added KR9: ~, OpenA3XX:Korry Switch, F.Cu at (296.9, 169.9)
- added P1: DataIn, Connector_PinHeader_2.54mm:PinHeader_1x04_P2.54mm_Vertical, B.Cu at (343.0, 98.0)
- added P2: Conn_01x02, TerminalBlock:TerminalBlock_bornier-2_P5.08mm, B.Cu at (349.4, 99.3)
- added R2: Iset, Resistor_THT:R_Axial_DIN0207_L6.3mm_D2.5mm_P10.16mm_Horizontal, B.Cu at (215.7, 142.5)
- added S6: LEDDSP3_CA, OpenA3XX:Disp7s3x_036, F.Cu at (150.8, 119.6)
- added S7: LEDDSP3_CA, OpenA3XX:Disp7s3x_036, F.Cu at (244.2, 119.6)
- added bottom: LOGO, OpenA3XX:OpenA3XXLogoSmall, B.Cu at (347.6, 124.0)
- added top: LOGO, OpenA3XX:OpenA3XXLogoSmall, F.Cu at (347.4, 124.0)
Other:
- board text added: "Flight Simulation Only"
- board text added: "https://www.github.com/OpenA3XX - ELEC V1.0"
- board text added: "© 2025 OpenA3XX • CC BY-SA 4.0"

Commit message: Iteration1 Elec Panel PCB Completed
Parts:
- added D10: LED, OpenA3XX:LED_Everlight-SMD3528_3.5x2.8mm_67-21ST, F.Cu at (62.0, 171.5)
- added D11: LED, OpenA3XX:LED_Everlight-SMD3528_3.5x2.8mm_67-21ST, F.Cu at (63.9, 186.5)
- added D12: LED, OpenA3XX:LED_Everlight-SMD3528_3.5x2.8mm_67-21ST, F.Cu at (82.2, 194.6)
- added D13: LED, OpenA3XX:LED_Everlight-SMD3528_3.5x2.8mm_67-21ST, F.Cu at (97.2, 187.9)
- added D14: LED, OpenA3XX:LED_Everlight-SMD3528_3.5x2.8mm_67-21ST, F.Cu at (96.9, 171.1)
- added D15: LED, OpenA3XX:LED_Everlight-SMD3528_3.5x2.8mm_67-21ST, F.Cu at (89.0, 162.2)
- added D16: LED, OpenA3XX:LED_Everlight-SMD3528_3.5x2.8mm_67-21ST, F.Cu at (96.9, 157.8)
- added D17: LED, OpenA3XX:LED_Everlight-SMD3528_3.5x2.8mm_67-21ST, F.Cu at (96.1, 135.7)
- added D18: LED, OpenA3XX:LED_Everlight-SMD3528_3.5x2.8mm_67-21ST, F.Cu at (97.2, 124.5)
- added D19: LED, OpenA3XX:LED_Everlight-SMD3528_3.5x2.8mm_67-21ST, F.Cu at (104.4, 113.3)
- added D2: LED, OpenA3XX:LED_Everlight-SMD3528_3.5x2.8mm_67-21ST, F.Cu at (66.5, 102.1)
- added D20: LED, OpenA3XX:LED_Everlight-SMD3528_3.5x2.8mm_67-21ST, F.Cu at (120.9, 113.4)
- added D21: LED, OpenA3XX:LED_Everlight-SMD3528_3.5x2.8mm_67-21ST, F.Cu at (107.8, 128.4)
- added D22: LED, OpenA3XX:LED_Everlight-SMD3528_3.5x2.8mm_67-21ST, F.Cu at (119.8, 142.6)
- added D23: LED, OpenA3XX:LED_Everlight-SMD3528_3.5x2.8mm_67-21ST, F.Cu at (108.3, 157.7)
- added D24: LED, OpenA3XX:LED_Everlight-SMD3528_3.5x2.8mm_67-21ST, F.Cu at (127.0, 166.2)
- added D25: LED, OpenA3XX:LED_Everlight-SMD3528_3.5x2.8mm_67-21ST, F.Cu at (128.4, 182.2)
- added D26: LED, OpenA3XX:LED_Everlight-SMD3528_3.5x2.8mm_67-21ST, F.Cu at (113.9, 194.8)
- added D27: LED, OpenA3XX:LED_Everlight-SMD3528_3.5x2.8mm_67-21ST, F.Cu at (141.9, 159.9)
- added D28: LED, OpenA3XX:LED_Everlight-SMD3528_3.5x2.8mm_67-21ST, F.Cu at (141.7, 132.8)
- added D29: LED, OpenA3XX:LED_Everlight-SMD3528_3.5x2.8mm_67-21ST, F.Cu at (163.8, 139.6)
- added D3: LED, OpenA3XX:LED_Everlight-SMD3528_3.5x2.8mm_67-21ST, F.Cu at (80.5, 98.8)
- added D30: LED, OpenA3XX:LED_Everlight-SMD3528_3.5x2.8mm_67-21ST, F.Cu at (162.2, 117.5)
- added D31: LED, OpenA3XX:LED_Everlight-SMD3528_3.5x2.8mm_67-21ST, F.Cu at (151.2, 106.3)
- added D32: LED, OpenA3XX:LED_Everlight-SMD3528_3.5x2.8mm_67-21ST, F.Cu at (166.9, 154.2)
- added D33: LED, OpenA3XX:LED_Everlight-SMD3528_3.5x2.8mm_67-21ST, F.Cu at (156.8, 166.3)
- added D34: LED, OpenA3XX:LED_Everlight-SMD3528_3.5x2.8mm_67-21ST, F.Cu at (155.0, 180.7)
- added D35: LED, OpenA3XX:LED_Everlight-SMD3528_3.5x2.8mm_67-21ST, F.Cu at (160.9, 194.8)
- added D36: LED, OpenA3XX:LED_Everlight-SMD3528_3.5x2.8mm_67-21ST, F.Cu at (182.9, 194.5)
- added D37: LED, OpenA3XX:LED_Everlight-SMD3528_3.5x2.8mm_67-21ST, F.Cu at (140.1, 195.1)
- added D38: LED, OpenA3XX:LED_Everlight-SMD3528_3.5x2.8mm_67-21ST, F.Cu at (187.5, 186.1)
- added D39: LED, OpenA3XX:LED_Everlight-SMD3528_3.5x2.8mm_67-21ST, F.Cu at (216.1, 194.8)
- added D4: LED, OpenA3XX:LED_Everlight-SMD3528_3.5x2.8mm_67-21ST, F.Cu at (96.8, 102.2)
- added D40: LED, OpenA3XX:LED_Everlight-SMD3528_3.5x2.8mm_67-21ST, F.Cu at (196.7, 176.4)
- added D41: LED, OpenA3XX:LED_Everlight-SMD3528_3.5x2.8mm_67-21ST, F.Cu at (184.8, 166.7)
- added D42: LED, OpenA3XX:LED_Everlight-SMD3528_3.5x2.8mm_67-21ST, F.Cu at (195.3, 160.8)
- added D43: LED, OpenA3XX:LED_Everlight-SMD3528_3.5x2.8mm_67-21ST, F.Cu at (193.4, 154.3)
- added D44: LED, OpenA3XX:LED_Everlight-SMD3528_3.5x2.8mm_67-21ST, F.Cu at (183.2, 132.9)
- added D45: LED, OpenA3XX:LED_Everlight-SMD3528_3.5x2.8mm_67-21ST, F.Cu at (170.1, 118.9)
- added D46: LED, OpenA3XX:LED_Everlight-SMD3528_3.5x2.8mm_67-21ST, F.Cu at (182.3, 103.8)
- added D47: LED, OpenA3XX:LED_Everlight-SMD3528_3.5x2.8mm_67-21ST, F.Cu at (213.5, 103.6)
- added D48: LED, OpenA3XX:LED_Everlight-SMD3528_3.5x2.8mm_67-21ST, F.Cu at (225.4, 119.5)
- added D49: LED, OpenA3XX:LED_Everlight-SMD3528_3.5x2.8mm_67-21ST, F.Cu at (244.8, 106.7)
- added D5: LED, OpenA3XX:LED_Everlight-SMD3528_3.5x2.8mm_67-21ST, F.Cu at (65.4, 116.0)
- added D50: LED, OpenA3XX:LED_Everlight-SMD3528_3.5x2.8mm_67-21ST, F.Cu at (201.0, 142.1)
- added D51: LED, OpenA3XX:LED_Everlight-SMD3528_3.5x2.8mm_67-21ST, F.Cu at (225.5, 142.9)
- added D52: LED, OpenA3XX:LED_Everlight-SMD3528_3.5x2.8mm_67-21ST, F.Cu at (247.9, 132.8)
- added D53: LED, OpenA3XX:LED_Everlight-SMD3528_3.5x2.8mm_67-21ST, F.Cu at (229.7, 153.8)
- added D54: LED, OpenA3XX:LED_Everlight-SMD3528_3.5x2.8mm_67-21ST, F.Cu at (226.5, 176.7)
- added D55: LED, OpenA3XX:LED_Everlight-SMD3528_3.5x2.8mm_67-21ST, F.Cu at (236.4, 184.3)
- added D56: LED, OpenA3XX:LED_Everlight-SMD3528_3.5x2.8mm_67-21ST, F.Cu at (252.8, 195.2)
- added D57: LED, OpenA3XX:LED_Everlight-SMD3528_3.5x2.8mm_67-21ST, F.Cu at (252.5, 153.4)
- added D58: LED, OpenA3XX:LED_Everlight-SMD3528_3.5x2.8mm_67-21ST, F.Cu at (256.2, 117.9)
- added D59: LED, OpenA3XX:LED_Everlight-SMD3528_3.5x2.8mm_67-21ST, F.Cu at (262.7, 140.7)
- added D6: LED, OpenA3XX:LED_Everlight-SMD3528_3.5x2.8mm_67-21ST, F.Cu at (59.2, 125.8)
- added D60: LED, OpenA3XX:LED_Everlight-SMD3528_3.5x2.8mm_67-21ST, F.Cu at (279.3, 145.9)
- added D61: LED, OpenA3XX:LED_Everlight-SMD3528_3.5x2.8mm_67-21ST, F.Cu at (280.0, 160.7)
- added D62: LED, OpenA3XX:LED_Everlight-SMD3528_3.5x2.8mm_67-21ST, F.Cu at (269.0, 171.7)
- added D63: LED, OpenA3XX:LED_Everlight-SMD3528_3.5x2.8mm_67-21ST, F.Cu at (238.1, 165.6)
- added D64: LED, OpenA3XX:LED_Everlight-SMD3528_3.5x2.8mm_67-21ST, F.Cu at (269.0, 185.6)
- added D65: LED, OpenA3XX:LED_Everlight-SMD3528_3.5x2.8mm_67-21ST, F.Cu at (290.4, 193.5)
- added D66: LED, OpenA3XX:LED_Everlight-SMD3528_3.5x2.8mm_67-21ST, F.Cu at (290.7, 168.6)
- added D67: LED, OpenA3XX:LED_Everlight-SMD3528_3.5x2.8mm_67-21ST, F.Cu at (302.4, 153.7)
- added D68: LED, OpenA3XX:LED_Everlight-SMD3528_3.5x2.8mm_67-21ST, F.Cu at (301.9, 142.8)
- added D69: LED, OpenA3XX:LED_Everlight-SMD3528_3.5x2.8mm_67-21ST, F.Cu at (294.0, 124.0)
- added D7: LED, OpenA3XX:LED_Everlight-SMD3528_3.5x2.8mm_67-21ST, F.Cu at (67.3, 131.9)
- added D70: LED, OpenA3XX:LED_Everlight-SMD3528_3.5x2.8mm_67-21ST, F.Cu at (278.2, 112.7)
- added D71: LED, OpenA3XX:LED_Everlight-SMD3528_3.5x2.8mm_67-21ST, F.Cu at (300.6, 113.4)
- added D72: LED, OpenA3XX:LED_Everlight-SMD3528_3.5x2.8mm_67-21ST, F.Cu at (316.6, 113.7)
- added D73: LED, OpenA3XX:LED_Everlight-SMD3528_3.5x2.8mm_67-21ST, F.Cu at (320.3, 128.6)
- added D74: LED, OpenA3XX:LED_Everlight-SMD3528_3.5x2.8mm_67-21ST, F.Cu at (317.3, 151.1)
- added D75: LED, OpenA3XX:LED_Everlight-SMD3528_3.5x2.8mm_67-21ST, F.Cu at (322.7, 168.4)
- added D76: LED, OpenA3XX:LED_Everlight-SMD3528_3.5x2.8mm_67-21ST, F.Cu at (323.0, 193.2)
- added D77: LED, OpenA3XX:LED_Everlight-SMD3528_3.5x2.8mm_67-21ST, F.Cu at (354.1, 193.2)
- added D78: LED, OpenA3XX:LED_Everlight-SMD3528_3.5x2.8mm_67-21ST, F.Cu at (354.6, 169.8)
- added D79: LED, OpenA3XX:LED_Everlight-SMD3528_3.5x2.8mm_67-21ST, F.Cu at (337.7, 157.6)
- added D8: LED, OpenA3XX:LED_Everlight-SMD3528_3.5x2.8mm_67-21ST, F.Cu at (63.7, 145.2)
- added D80: LED, OpenA3XX:LED_Everlight-SMD3528_3.5x2.8mm_67-21ST, F.Cu at (365.6, 179.5)
- added D81: LED, OpenA3XX:LED_Everlight-SMD3528_3.5x2.8mm_67-21ST, F.Cu at (363.1, 157.8)
- added D82: LED, OpenA3XX:LED_Everlight-SMD3528_3.5x2.8mm_67-21ST, F.Cu at (361.9, 135.0)
- added D83: LED, OpenA3XX:LED_Everlight-SMD3528_3.5x2.8mm_67-21ST, F.Cu at (366.7, 119.8)
- added D84: LED, OpenA3XX:LED_Everlight-SMD3528_3.5x2.8mm_67-21ST, F.Cu at (326.6, 141.1)
- added D9: LED, OpenA3XX:LED_Everlight-SMD3528_3.5x2.8mm_67-21ST, F.Cu at (64.0, 159.6)
- added R10: 220R, Resistor_SMD:R_1206_3216Metric_Pad1.30x1.75mm_HandSolder, F.Cu at (141.8, 140.8)
- added R11: 220R, Resistor_SMD:R_1206_3216Metric_Pad1.30x1.75mm_HandSolder, F.Cu at (144.0, 106.4)
- added R12: 220R, Resistor_SMD:R_1206_3216Metric_Pad1.30x1.75mm_HandSolder, F.Cu at (154.7, 188.4)
- added R13: 220R, Resistor_SMD:R_1206_3216Metric_Pad1.30x1.75mm_HandSolder, F.Cu at (172.0, 194.7)
- added R14: 220R, Resistor_SMD:R_1206_3216Metric_Pad1.30x1.75mm_HandSolder, F.Cu at (187.4, 176.0)
- added R15: 220R, Resistor_SMD:R_1206_3216Metric_Pad1.30x1.75mm_HandSolder, F.Cu at (184.7, 160.5)
- added R16: 220R, Resistor_SMD:R_1206_3216Metric_Pad1.30x1.75mm_HandSolder, F.Cu at (155.3, 139.4)
- added R17: 220R, Resistor_SMD:R_1206_3216Metric_Pad1.30x1.75mm_HandSolder, F.Cu at (165.4, 106.2)
- added R18: 220R, Resistor_SMD:R_1206_3216Metric_Pad1.30x1.75mm_HandSolder, F.Cu at (227.6, 106.0)
- added R19: 220R, Resistor_SMD:R_1206_3216Metric_Pad1.30x1.75mm_HandSolder, F.Cu at (234.0, 146.3)
- added R2: 220R, Resistor_SMD:R_1206_3216Metric_Pad1.30x1.75mm_HandSolder, F.Cu at (97.4, 114.2)
- added R20: 220R, Resistor_SMD:R_1206_3216Metric_Pad1.30x1.75mm_HandSolder, F.Cu at (236.4, 192.7)
- added R21: 220R, Resistor_SMD:R_1206_3216Metric_Pad1.30x1.75mm_HandSolder, F.Cu at (260.4, 153.2)
- added R22: 220R, Resistor_SMD:R_1206_3216Metric_Pad1.30x1.75mm_HandSolder, F.Cu at (287.2, 145.9)
- added R23: 220R, Resistor_SMD:R_1206_3216Metric_Pad1.30x1.75mm_HandSolder, F.Cu at (240.9, 153.4)
- added R24: 220R, Resistor_SMD:R_1206_3216Metric_Pad1.30x1.75mm_HandSolder, F.Cu at (290.1, 176.3)
- added R25: 220R, Resistor_SMD:R_1206_3216Metric_Pad1.30x1.75mm_HandSolder, F.Cu at (301.6, 128.8)
- added R26: 220R, Resistor_SMD:R_1206_3216Metric_Pad1.30x1.75mm_HandSolder, F.Cu at (317.0, 120.5)
- added R27: 220R, Resistor_SMD:R_1206_3216Metric_Pad1.30x1.75mm_HandSolder, F.Cu at (327.7, 160.8)
- added R28: 220R, Resistor_SMD:R_1206_3216Metric_Pad1.30x1.75mm_HandSolder, F.Cu at (355.1, 177.7)
- added R29: 220R, Resistor_SMD:R_1206_3216Metric_Pad1.30x1.75mm_HandSolder, F.Cu at (355.6, 157.6)
- added R3: 220R, Resistor_SMD:R_1206_3216Metric_Pad1.30x1.75mm_HandSolder, F.Cu at (63.6, 137.8)
- added R30: 220R, Resistor_SMD:R_1206_3216Metric_Pad1.30x1.75mm_HandSolder, F.Cu at (334.7, 140.8)
- added R4: 220R, Resistor_SMD:R_1206_3216Metric_Pad1.30x1.75mm_HandSolder, F.Cu at (72.4, 162.2)
- added R5: 220R, Resistor_SMD:R_1206_3216Metric_Pad1.30x1.75mm_HandSolder, F.Cu at (97.2, 194.4)
- added R6: 220R, Resistor_SMD:R_1206_3216Metric_Pad1.30x1.75mm_HandSolder, F.Cu at (101.2, 150.4)
- added R7: 220R, Resistor_SMD:R_1206_3216Metric_Pad1.30x1.75mm_HandSolder, F.Cu at (105.0, 121.2)
- added R8: 220R, Resistor_SMD:R_1206_3216Metric_Pad1.30x1.75mm_HandSolder, F.Cu at (119.8, 150.3)
- added R9: 220R, Resistor_SMD:R_1206_3216Metric_Pad1.30x1.75mm_HandSolder, F.Cu at (128.6, 189.2)
- moved J1 70.0 mm to (130.3, 99.1)
- moved S1 4.00 mm to (146.8, 119.6)
- moved S2 3.39 mm to (240.8, 119.6)
- renumbered C2 to C1, C3 to C2, J21 to J1, J1 to J2, P2 to P1, P1 to P2, R2 to R1, S6 to S1, S7 to S2
Connections:
- S1 pad 12: /A5 -> /A2
- S1 pad 8: /A3 -> /A0
- S1 pad 9: /A4 -> /A1
- S2 pad 12: /A2 -> /A5
- S2 pad 8: /A0 -> /A3
- S2 pad 9: /A1 -> /A4
Routing:
- net GND: track 0.00 -> 1247.3 mm, vias 0 -> 13
- net +12V: track 0.00 -> 922.5 mm, vias 0 -> 22
- net Net-(J2-Pin_6): track 0.00 -> 326.7 mm, vias 0 -> 1
- net Net-(J2-Pin_5): track 0.00 -> 308.5 mm, vias 0 -> 1
- net Net-(J2-Pin_4): track 0.00 -> 307.6 mm, vias 0 -> 1
- net Net-(J2-Pin_18): track 0.00 -> 281.8 mm, vias 0 -> 3
- net Net-(J2-Pin_21): track 0.00 -> 267.3 mm, vias 0 -> 2
- net Net-(J2-Pin_16): track 0.00 -> 265.4 mm, vias 0 -> 2
- net Net-(J2-Pin_3): track 0.00 -> 261.9 mm, vias 0 -> 2
- net Net-(J2-Pin_2): track 0.00 -> 260.0 mm, vias 0 -> 1
- net Net-(J2-Pin_20): track 0.00 -> 259.9 mm, vias 0 -> 1
- net Net-(J2-Pin_17): track 0.00 -> 259.9 mm, vias 0 -> 1
- net Net-(J2-Pin_19): track 0.00 -> 258.0 mm, vias 0 -> 1
- net Net-(J2-Pin_1): track 0.00 -> 244.2 mm
- net Net-(J2-Pin_9): track 0.00 -> 230.7 mm, vias 0 -> 2
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