File: overhead/elec/electronics/elec.kicad_sch (KiCad schematic)
At the start: 0 parts

Commit message: Elec PCB continuation
Parts:
- added C2: 10uF, Capacitor_THT:CP_Radial_D5.0mm_P2.50mm, symbol GCC_device:CP
- added C3: 0.1 uF, Capacitor_SMD:C_1206_3216Metric_Pad1.33x1.80mm_HandSolder, symbol GCC_device:C
- added D1: 1N5818, Diode_SMD:D_SMA_Handsoldering, symbol Device:D_Schottky_ALT
- added IC1: MAX7219CWG, Package_SO:SOIC-24W_7.5x15.4mm_P1.27mm, symbol GCC_drivers:MAX7219CNG
- added J1: Conn_02x20_Counter_Clockwise, Connector_PinHeader_2.54mm:PinHeader_2x20_P2.54mm_Vertical, symbol Connector_Generic:Conn_02x20_Counter_Clockwise
- added J21: Conn_02x01, TerminalBlock:TerminalBlock_bornier-2_P5.08mm, symbol Connector_Generic:Conn_02x01
- added KR1, KR10, KR11, KR12, KR2, KR3, KR4, KR5, KR6, KR7, KR8, KR9: ~, OpenA3XX:Korry Switch, symbol KorrySwitch:Korry_Switch
- added P1: DataIn, Connector_PinHeader_2.54mm:PinHeader_1x04_P2.54mm_Vertical, symbol Connector_Generic:Conn_01x04
- added P2: Conn_01x02, TerminalBlock:TerminalBlock_bornier-2_P5.08mm, symbol Connector_Generic:Conn_01x02
- added R2: Iset, Resistor_THT:R_Axial_DIN0207_L6.3mm_D2.5mm_P10.16mm_Horizontal, symbol GCC_device:R
- added S6, S7: LEDDSP3_CA, OpenA3XX:Disp7s3x_036, symbol GCC_display:LEDDSP3_CA
Connections:
- new net: IC1.18 (ISET), R2.2
- new net: J1.31 (Pin_31), KR11.1 (+5V_TOP_LED)
- new net: J1.32 (Pin_32), KR11.3 (+5V_BOTTOM_LED)
- new net: J1.33 (Pin_33), KR11.5 (SW_IN)
- new net: J1.19 (Pin_19), KR4.1 (+5V_TOP_LED)
- new net: J1.20 (Pin_20), KR4.3 (+5V_BOTTOM_LED)
- new net: J1.21 (Pin_21), KR4.5 (SW_IN)
- new net: J1.1 (Pin_1), KR1.1 (+5V_TOP_LED)
- new net: J1.10 (Pin_10), KR7.1 (+5V_TOP_LED)
- new net: J1.11 (Pin_11), KR7.3 (+5V_BOTTOM_LED)
- new net: J1.12 (Pin_12), KR7.5 (SW_IN)
- new net: J1.13 (Pin_13), KR9.1 (+5V_TOP_LED)
- new net: J1.14 (Pin_14), KR9.3 (+5V_BOTTOM_LED)
- new net: J1.15 (Pin_15), KR9.5 (SW_IN)
- new net: J1.16 (Pin_16), KR2.1 (+5V_TOP_LED)
- new net: J1.17 (Pin_17), KR2.3 (+5V_BOTTOM_LED)
- new net: J1.18 (Pin_18), KR2.5 (SW_IN)
- new net: J1.2 (Pin_2), KR1.3 (+5V_BOTTOM_LED)
- new net: J1.22 (Pin_22), KR6.1 (+5V_TOP_LED)
- new net: J1.23 (Pin_23), KR6.3 (+5V_BOTTOM_LED)
- new net: J1.24 (Pin_24), KR8.1 (+5V_TOP_LED)
- new net: J1.25 (Pin_25), KR6.5 (SW_IN)
- new net: J1.26 (Pin_26), KR8.3 (+5V_BOTTOM_LED)
- new net: J1.27 (Pin_27), KR8.5 (SW_IN)
- new net: J1.28 (Pin_28), KR10.1 (+5V_TOP_LED)
- new net: J1.29 (Pin_29), KR10.3 (+5V_BOTTOM_LED)
- new net: J1.3 (Pin_3), KR1.5 (SW_IN)
- new net: J1.30 (Pin_30), KR10.5 (SW_IN)
- new net: J1.34 (Pin_34), KR12.1 (+5V_TOP_LED)
- new net: J1.35 (Pin_35), KR12.3 (+5V_BOTTOM_LED)
- new net: J1.36 (Pin_36), KR12.5 (SW_IN)
- new net: J1.4 (Pin_4), KR3.1 (+5V_TOP_LED)
- new net: J1.5 (Pin_5), KR3.3 (+5V_BOTTOM_LED)
- new net: J1.6 (Pin_6), KR3.5 (SW_IN)
- new net: J1.7 (Pin_7), KR5.1 (+5V_TOP_LED)
- new net: J1.8 (Pin_8), KR5.3 (+5V_BOTTOM_LED)
- new net: J1.9 (Pin_9), KR5.5 (SW_IN)
- new net +12V: J21.2 (Pin_2)
- new net A0: IC1.2 (DIG0), S7.8 (A1)
- new net A1: IC1.11 (DIG1), S7.9 (A2)
- new net A2: IC1.6 (DIG2), S7.12 (A3)
- new net A3: IC1.7 (DIG3), S6.8 (A1)
- new net A4: IC1.3 (DIG4), S6.9 (A2)
- new net A5: IC1.10 (DIG5), S6.12 (A3)
- new net A_SegA: IC1.14 (SEGA), S6.11 (a), S7.11 (a)
- new net A_SegB: IC1.16 (SEGB), S6.7 (b), S7.7 (b)
- new net A_SegC: IC1.20 (SEGC), S6.4 (c), S7.4 (c)
- new net A_SegD: IC1.23 (SEGD), S6.2 (d), S7.2 (d)
- new net A_SegDP: IC1.22 (SEGDP), S6.3 (dp), S7.3 (dp)
- new net A_SegE: IC1.21 (SEGE), S6.1 (e), S7.1 (e)
- new net A_SegF: IC1.15 (SEGF), S6.10 (f), S7.10 (f)
- new net A_SegG: IC1.17 (SEGG), S6.5 (g), S7.5 (g)
- new net Clk: IC1.13 (CLK), P1.4 (Pin_4)
- new net Din: IC1.1 (DIN), P1.2 (Pin_2)
- new net GND: C2.2, C3.2, IC1.4 (GND1), IC1.9 (GND2), J21.1 (Pin_1), KR1.2 (GND_TOP_LED), KR1.4 (GND_BOTTOM_LED), KR1.6 (SW_OUT), KR10.2 (GND_TOP_LED), KR10.4 (GND_BOTTOM_LED), KR10.6 (SW_OUT), KR11.2 (GND_TOP_LED), KR11.4 (GND_BOTTOM_LED), KR11.6 (SW_OUT), KR12.2 (GND_TOP_LED), KR12.4 (GND_BOTTOM_LED), KR12.6 (SW_OUT), KR2.2 (GND_TOP_LED), KR2.4 (GND_BOTTOM_LED), KR2.6 (SW_OUT), KR3.2 (GND_TOP_LED), KR3.4 (GND_BOTTOM_LED), KR3.6 (SW_OUT), KR4.2 (GND_TOP_LED), KR4.4 (GND_BOTTOM_LED), KR4.6 (SW_OUT), KR5.2 (GND_TOP_LED), KR5.4 (GND_BOTTOM_LED), KR5.6 (SW_OUT), KR6.2 (GND_TOP_LED), KR6.4 (GND_BOTTOM_LED), KR6.6 (SW_OUT), KR7.2 (GND_TOP_LED), KR7.4 (GND_BOTTOM_LED), KR7.6 (SW_OUT), KR8.2 (GND_TOP_LED), KR8.4 (GND_BOTTOM_LED), KR8.6 (SW_OUT), KR9.2 (GND_TOP_LED), KR9.4 (GND_BOTTOM_LED), KR9.6 (SW_OUT), P1.1 (Pin_1), P2.2 (Pin_2)
- new net K6: IC1.5 (DIG6)
- new net K7: IC1.8 (DIG7)
- new net Sel: IC1.12 (LOAD), P1.3 (Pin_3)
- new net Vcc: C2.1, C3.1, D1.1 (K), IC1.19 (VCC), R2.1
- new net Vin: D1.2 (A), P2.1 (Pin_1)
- no-connect marks 0 -> 3

Commit message: Iteration1 Elec Panel PCB Completed
Parts:
- added D10, D11, D12, D13, D14, D15, D16, D17, D18, D19, D2, D20, D21, D22, D23, D24, D25, D26, D27, D28, D29, D3, D30, D31, D32, D33, D34, D35, D36, D37, D38, D39, D4, D40, D41, D42, D43, D44, D45, D46, D47, D48, D49, D5, D50, D51, D52, D53, D54, D55, D56, D57, D58, D59, D6, D60, D61, D62, D63, D64, D65, D66, D67, D68, D69, D7, D70, D71, D72, D73, D74, D75, D76, D77, D78, D79, D8, D80, D81, D82, D83, D84, D9: LED, OpenA3XX:LED_Everlight-SMD3528_3.5x2.8mm_67-21ST, symbol Device:LED
- added R10, R11, R12, R13, R14, R15, R16, R17, R18, R19, R2, R20, R21, R22, R23, R24, R25, R26, R27, R28, R29, R3, R30, R4, R5, R6, R7, R8, R9: 220R, Resistor_SMD:R_1206_3216Metric_Pad1.30x1.75mm_HandSolder, symbol Device:R
- renumbered C2 to C1, C3 to C2, J21 to J1, J1 to J2, P2 to P1, P1 to P2, R2 to R1, S7 to S1, S6 to S2
Connections:
- net +12V: now also D11.2 (A), D14.2 (A), D17.2 (A), D2.2 (A), D20.2 (A), D23.2 (A), D26.2 (A), D29.2 (A), D32.2 (A), D35.2 (A), D36.2 (A), D39.2 (A), D42.2 (A), D45.2 (A), D46.2 (A), D49.2 (A), D5.2 (A), D52.2 (A), D55.2 (A), D58.2 (A), D61.2 (A), D64.2 (A), D67.2 (A), D70.2 (A), D73.2 (A), D76.2 (A), D79.2 (A), D8.2 (A), D82.2 (A)
- net GND: now also R10.2, R11.2, R12.2, R13.2, R14.2, R15.2, R16.2, R17.2, R18.2, R19.2, R2.2, R20.2, R21.2, R22.2, R23.2, R24.2, R25.2, R26.2, R27.2, R28.2, R29.2, R3.2, R30.2, R4.2, R5.2, R6.2, R7.2, R8.2, R9.2
- new net: D66.1 (K), R24.1
- new net: D63.1 (K), R23.1
- new net: D43.1 (K), D44.2 (A)
- new net: D42.1 (K), D43.2 (A)
- new net: D3.1 (K), D4.2 (A)
- new net: D2.1 (K), D3.2 (A)
- new net: D25.1 (K), R9.1
- new net: D18.1 (K), D19.2 (A)
- new net: D17.1 (K), D18.2 (A)
- new net: D75.1 (K), R27.1
- new net: D74.1 (K), D75.2 (A)
- new net: D26.1 (K), D27.2 (A)
- new net: D19.1 (K), R7.1
- new net: D51.1 (K), R19.1
- new net: D35.1 (K), R13.1
- new net: D56.1 (K), D57.2 (A)
- new net: D55.1 (K), D56.2 (A)
- new net: D69.1 (K), R25.1
- new net: D68.1 (K), D69.2 (A)
- new net: D16.1 (K), R6.1
- new net: D73.1 (K), D74.2 (A)
- new net: D70.1 (K), D71.2 (A)
- new net: D78.1 (K), R28.1
- new net: D46.1 (K), D47.2 (A)
- new net: D4.1 (K), R2.1
- new net: D62.1 (K), D63.2 (A)
- new net: D61.1 (K), D62.2 (A)
- new net: D47.1 (K), D48.2 (A)
- new net: D84.1 (K), R30.1
- new net: D71.1 (K), D72.2 (A)
- new net: D8.1 (K), D9.2 (A)
- new net: D45.1 (K), R17.1
- new net: D10.1 (K), R4.1
- new net: D21.1 (K), D22.2 (A)
- new net: D20.1 (K), D21.2 (A)
- new net: D67.1 (K), D68.2 (A)
- new net: D65.1 (K), D66.2 (A)
- new net: D64.1 (K), D65.2 (A)
- new net: D34.1 (K), R12.1
- new net: D14.1 (K), D15.2 (A)
- new net: D60.1 (K), R22.1
- new net: D59.1 (K), D60.2 (A)
- new net: D29.1 (K), D30.2 (A)
- new net: D48.1 (K), R18.1
- new net: D57.1 (K), R21.1
- new net: D36.1 (K), D37.2 (A)
- new net: D50.1 (K), D51.2 (A)
- new net: D49.1 (K), D50.2 (A)
- new net: D58.1 (K), D59.2 (A)
- new net: D31.1 (K), R11.1
- new net: D30.1 (K), D31.2 (A)
- new net: D13.1 (K), R5.1
- new net: D12.1 (K), D13.2 (A)
- new net: D5.1 (K), D6.2 (A)
- new net: D77.1 (K), D78.2 (A)
- new net: D10.2 (A), D9.1 (K)
- new net: D38.1 (K), R14.1
- new net: D37.1 (K), D38.2 (A)
- new net: D54.1 (K), R20.1
- new net: D53.1 (K), D54.2 (A)
- new net: D22.1 (K), R8.1
- new net: D72.1 (K), R26.1
- new net: D76.1 (K), D77.2 (A)
- new net: D24.1 (K), D25.2 (A)
- new net: D33.1 (K), D34.2 (A)
- new net: D32.1 (K), D33.2 (A)
- new net: D79.1 (K), D80.2 (A)
- new net: D82.1 (K), D83.2 (A)
- new net: D41.1 (K), R15.1
- new net: D28.1 (K), R10.1
- new net: D7.1 (K), R3.1
- new net: D6.1 (K), D7.2 (A)
- new net: D15.1 (K), D16.2 (A)
- new net: D27.1 (K), D28.2 (A)
- new net: D40.1 (K), D41.2 (A)
- new net: D39.1 (K), D40.2 (A)
- new net: D23.1 (K), D24.2 (A)
- new net: D44.1 (K), R16.1
- new net: D83.1 (K), D84.2 (A)
- new net: D11.1 (K), D12.2 (A)
- new net: D52.1 (K), D53.2 (A)
- new net: D81.1 (K), R29.1
- new net: D80.1 (K), D81.2 (A)
