File: overhead/left/adirs/electronics/adirs.kicad_sch (KiCad schematic)
At the start: 67 parts, among them J1 Conn_02x01, J2 Conn_02x13_Counter_Clockwise, J3 Conn_02x01, J4 Conn_02x02_Counter_Clockwise, J5 Conn_02x02_Counter_Clockwise, J6 Conn_02x02_Counter_Clockwise

Commit message: ADIRS - Iteration 2 - Completed
Parts:
- removed J2: Conn_02x13_Counter_Clockwise, Connector_PinHeader_2.54mm:PinHeader_2x14_P2.54mm_Vertical, symbol Connector_Generic:Conn_02x14_Counter_Clockwise
- added J2: Conn_02x20_Counter_Clockwise, Connector_PinHeader_2.54mm:PinHeader_2x20_P2.54mm_Vertical, symbol Connector_Generic:Conn_02x20_Counter_Clockwise
- added J7: Conn_02x01, TerminalBlock:TerminalBlock_bornier-2_P5.08mm, symbol Connector_Generic:Conn_02x01
Connections:
- net +12V: now also J7.2 (Pin_2)
- net GND: now also J7.1 (Pin_1)
- net at J4.2 (Pin_2): now also J2.20 (Pin_20)
- net at J4.3 (Pin_3): now also J2.21 (Pin_21)
- net at J4.4 (Pin_4): now also J2.22 (Pin_22)
- net at KR4.1 (+5V_TOP_LED): now also J2.13 (Pin_13)
- net at KR4.3 (+5V_BOTTOM_LED): now also J2.14 (Pin_14)
- net at KR4.5 (SW_IN): now also J2.15 (Pin_15)
- net at J3.2 (Pin_2): now also J2.19 (Pin_19)
- net at J6.2 (Pin_2): now also J2.26 (Pin_26)
- net at J6.3 (Pin_3): now also J2.27 (Pin_27)
- net at J6.4 (Pin_4): now also J2.28 (Pin_28)
- net at KR1.1 (+5V_TOP_LED): now also J2.1 (Pin_1)
- net at KR2.1 (+5V_TOP_LED): now also J2.10 (Pin_10)
- net at KR2.3 (+5V_BOTTOM_LED): now also J2.11 (Pin_11)
- net at KR2.5 (SW_IN): now also J2.12 (Pin_12)
- net at KR6.1 (+5V_TOP_LED): now also J2.16 (Pin_16)
- net at KR6.3 (+5V_BOTTOM_LED): now also J2.17 (Pin_17)
- net at KR6.5 (SW_IN): now also J2.18 (Pin_18)
- net at KR1.3 (+5V_BOTTOM_LED): now also J2.2 (Pin_2)
- net at J5.2 (Pin_2): now also J2.23 (Pin_23)
- net at J5.3 (Pin_3): now also J2.24 (Pin_24)
- net at J5.4 (Pin_4): now also J2.25 (Pin_25)
- net at KR1.5 (SW_IN): now also J2.3 (Pin_3)
- net at KR3.1 (+5V_TOP_LED): now also J2.4 (Pin_4)
- net at KR3.3 (+5V_BOTTOM_LED): now also J2.5 (Pin_5)
- net at KR3.5 (SW_IN): now also J2.6 (Pin_6)
- net at KR5.1 (+5V_TOP_LED): now also J2.7 (Pin_7)
- net at KR5.3 (+5V_BOTTOM_LED): now also J2.8 (Pin_8)
- net at KR5.5 (SW_IN): now also J2.9 (Pin_9)
- no-connect marks 0 -> 12
