File: overhead/left/adirs/electronics/adirs.kicad_pcb (KiCad board)
At the start: 2 copper layers, 145 x 133 mm, 69 parts, among them J1 Conn_02x01, J2 Conn_02x13_Counter_Clockwise, J3 Conn_02x01, J4 Conn_02x02_Counter_Clockwise, J5 Conn_02x02_Counter_Clockwise, J6 Conn_02x02_Counter_Clockwise

Commit message: ADIRS - Iteration 2 - Completed
Parts:
- added J7: Conn_02x01, TerminalBlock:TerminalBlock_bornier-2_P5.08mm, B.Cu at (182.4, 150.4)
- J2: value Conn_02x13_Counter_Clockwise -> Conn_02x20_Counter_Clockwise; footprint Connector_PinHeader_2.54mm:PinHeader_2x14_P2.54mm_Vertical -> Connector_PinHeader_2.54mm:PinHeader_2x20_P2.54mm_Vertical
- moved J2 3.91 mm to (269.8, 28.5)
- moved R14 2.78 mm to (224.7, 33.4)
- moved J1 0.20 mm to (143.7, 25.4)
Routing:
- net Net-(J2-Pin_16): track 155.0 -> 105.4 mm, vias 2 -> 0
- net Net-(J2-Pin_18): track 162.6 -> 140.0 mm, vias 1 -> 4
- net Net-(J2-Pin_24): track 104.5 -> 83.9 mm, vias 1 -> 0
- net GND: track 724.2 -> 708.3 mm
- net +12V: track 518.9 -> 503.3 mm, vias 10 -> 11
- net Net-(J2-Pin_2): track 133.1 -> 148.0 mm, vias 2 -> 1
- net Net-(D28-K): track 49.5 -> 36.4 mm, vias 2 -> 0
- net Net-(J2-Pin_22): track 150.7 -> 161.5 mm
- net Net-(J2-Pin_7): track 151.1 -> 140.4 mm
- net Net-(J2-Pin_23): track 84.8 -> 74.7 mm, vias 1 -> 0
- net Net-(J2-Pin_8): track 169.7 -> 160.3 mm
- net Net-(J2-Pin_21): track 150.4 -> 159.6 mm, vias 2 -> 1
- net Net-(J2-Pin_6): track 70.4 -> 61.6 mm
- net Net-(J2-Pin_3): track 140.4 -> 133.5 mm, vias 2 -> 0
- net Net-(D8-K): track 41.3 -> 34.5 mm, vias 2 -> 0
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Other:
- board text added: "40"
- board text added: "https://www.github.com/OpenA3XX - ADIRS Panel V1.0"
- board text removed: "2"
- board text removed: "27"
- board text removed: "28"
- board text removed: "https://www.gitgub.com/OpenA3XX - ADIRS Panel V1.0"
