File: overhead/left/evac/electronics/evac.kicad_pcb (KiCad board)
At the start: 2 copper layers, 145 x 47.3 mm, 39 parts, among them J1 Conn_02x01, J2 Conn_02x01, J3 Conn_02x03_Counter_Clockwise, J4 Conn_02x01

Commit message: Gerber Files generation and updates
Parts:
- added J7: Conn_02x01, TerminalBlock:TerminalBlock_bornier-2_P5.08mm, B.Cu at (91.9, 121.8)
- J3: value Conn_02x03_Counter_Clockwise -> Conn_02x20_Counter_Clockwise; footprint Connector_PinHeader_2.54mm:PinHeader_2x03_P2.54mm_Vertical -> Connector_PinHeader_2.54mm:PinHeader_2x20_P2.54mm_Vertical
- J4: value Conn_02x01 -> Conn_01x03; footprint Connector_PinHeader_2.54mm:PinHeader_1x02_P2.54mm_Vertical -> Connector_PinHeader_2.54mm:PinHeader_1x03_P2.54mm_Vertical
- moved D6 4.51 mm to (167.2, 87.2)
- moved R2 3.49 mm to (175.3, 88.7)
- moved D20 2.93 mm to (189.6, 119.7)
- moved D11 2.43 mm to (197.2, 87.3)
- moved D10 1.78 mm to (184.0, 87.5)
- moved J3 1.38 mm to (214.7, 83.8)
- moved J4 0.92 mm to (187.1, 105.8)
- moved D5 0.59 mm to (146.5, 84.7)
Connections:
- J3 pad 6: unconnected-(J3-Pin_6-Pad6) -> Net-(J3-Pin_6)
- J4 pad 1: GND -> Net-(J3-Pin_5)
- J4 pad 2: Net-(J3-Pin_5) -> Net-(J3-Pin_6)
Routing:
- net GND: track 285.4 -> 337.0 mm
- net Net-(D18-K): track 24.3 -> 62.1 mm, vias 0 -> 2
- net +12V: track 227.5 -> 264.7 mm, vias 2 -> 4
- net Net-(J3-Pin_6): track 0.00 -> 33.9 mm
- net Net-(J3-Pin_2): track 97.0 -> 125.6 mm
- net Net-(J3-Pin_1): track 97.6 -> 109.9 mm
- net Net-(D22-K): track 62.2 -> 74.3 mm
- net Net-(D13-K): track 27.7 -> 36.4 mm
- net Net-(D3-K): track 24.0 -> 32.6 mm, vias 0 -> 2
- net Net-(D21-K): track 9.19 -> 17.1 mm
- net Net-(J3-Pin_3): track 123.1 -> 117.4 mm, vias 3 -> 1
- net Net-(D12-K): track 24.6 -> 30.2 mm
- net Net-(D19-K): track 20.6 -> 15.6 mm
- net Net-(J2-Pin_2): track 77.2 -> 80.6 mm
- net Net-(J3-Pin_5): track 28.6 -> 31.8 mm
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Other:
- board text added: "1-COMMAND-TOP_LED 2-COMMAND-BOTTOM_LED 3-COMMAND-KORRY_SW 4-HORN_SHUT_OFF_SW 5-CAPT_PURS_SW 6-CAPT_SW"
- board text added: "40"
- board text added: "https://www.github.com/OpenA3XX - EVAC Panel V1.0"
- board text removed: "1-COMMAND-TOP_LED 2-COMMAND-BOTTOM_LED 3-COMMAND-KORRY_SW 4-HORN_SHUT_OFF_SW 5-CAPT_PURS_SW"
- board text removed: "2"
- board text removed: "5"
- board text removed: "6"
- board text removed: "https://www.gitgub.com/OpenA3XX - EVAC Panel V1.0"
