File: overhead/left/evac/electronics/evac.kicad_sch (KiCad schematic)
At the start: 37 parts, among them J1 Conn_02x01, J2 Conn_02x01, J3 Conn_02x03_Counter_Clockwise, J4 Conn_02x01

Commit message: Gerber Files generation and updates
Parts:
- removed J3: Conn_02x03_Counter_Clockwise, Connector_PinHeader_2.54mm:PinHeader_2x03_P2.54mm_Vertical, symbol Connector_Generic:Conn_02x03_Counter_Clockwise
- removed J4: Conn_02x01, Connector_PinHeader_2.54mm:PinHeader_1x02_P2.54mm_Vertical, symbol Connector_Generic:Conn_02x01
- added J3: Conn_02x20_Counter_Clockwise, Connector_PinHeader_2.54mm:PinHeader_2x20_P2.54mm_Vertical, symbol Connector_Generic:Conn_02x20_Counter_Clockwise
- added J4: Conn_01x03, Connector_PinHeader_2.54mm:PinHeader_1x03_P2.54mm_Vertical, symbol Connector_Generic:Conn_01x03
- added J7: Conn_02x01, TerminalBlock:TerminalBlock_bornier-2_P5.08mm, symbol Connector_Generic:Conn_02x01
Connections:
- net +12V: now also J7.2 (Pin_2)
- net GND: now also J4.3 (Pin_3), J7.1 (Pin_1)
- net at KR1.1 (+5V_TOP_LED): now also J3.1 (Pin_1)
- net at KR1.3 (+5V_BOTTOM_LED): now also J3.2 (Pin_2)
- net at KR1.5 (SW_IN): now also J3.3 (Pin_3)
- net at J2.2 (Pin_2): now also J3.4 (Pin_4)
- new net: J3.5 (Pin_5), J4.1 (Pin_1)
- new net: J3.6 (Pin_6), J4.2 (Pin_2)
- no-connect marks 0 -> 34
Other:
- note added: "CAPT & PURS / CAPT"
- note added: "HORN SHUT OFF"
