File: overhead/left/flt-ctl/electronics/fl-ctl/fl-ctl.kicad_pcb (KiCad board)
At the start: 2 copper layers, 145 x 47.3 mm, 31 parts, among them J1 Conn_02x01, J2 Conn_02x05_Counter_Clockwise

Commit message: Gerber Files generation and updates
Parts:
- added J7: Conn_02x01, TerminalBlock:TerminalBlock_bornier-2_P5.08mm, B.Cu at (93.5, 120.2)
- J2: value Conn_02x05_Counter_Clockwise -> Conn_02x20_Counter_Clockwise; footprint Connector_PinHeader_2.54mm:PinHeader_2x05_P2.54mm_Vertical -> Connector_PinHeader_2.54mm:PinHeader_2x20_P2.54mm_Vertical
- moved D17 3.14 mm to (204.2, 119.3)
- moved D8 1.92 mm to (193.5, 85.5)
- moved D18 1.34 mm to (161.2, 119.1)
- moved D16 1.23 mm to (177.3, 118.7)
- moved R6 1.00 mm to (191.3, 119.0)
- moved R5 0.99 mm to (145.0, 119.0)
- moved D15 0.55 mm to (136.6, 119.5)
- moved D14 0.35 mm to (122.4, 119.5)
Routing:
- net GND: track 249.2 -> 302.8 mm
- net +12V: track 173.3 -> 213.5 mm, vias 3 -> 4
- net Net-(J2-Pin_6): track 113.5 -> 80.3 mm
- net Net-(D2-K): track 32.5 -> 16.8 mm, vias 2 -> 0
- net Net-(J2-Pin_8): track 42.3 -> 27.9 mm, vias 1 -> 0
- net Net-(D6-K): track 22.3 -> 8.03 mm, vias 2 -> 0
- net Net-(D4-K): track 31.4 -> 18.1 mm, vias 2 -> 0
- net Net-(J2-Pin_3): track 101.5 -> 113.0 mm
- net Net-(D5-K): track 14.4 -> 24.0 mm, vias 0 -> 2
- net Net-(J2-Pin_2): track 108.3 -> 99.0 mm, vias 2 -> 1
- net Net-(J2-Pin_4): track 56.7 -> 65.6 mm, vias 0 -> 1
- net Net-(J2-Pin_5): track 52.2 -> 60.5 mm, vias 1 -> 2
- net Net-(J2-Pin_9): track 30.4 -> 37.6 mm
- net Net-(J2-Pin_7): track 24.3 -> 30.6 mm
- net Net-(D11-K): track 42.3 -> 36.7 mm, vias 2 -> 0
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Other:
- board text added: "40"
- board text added: "https://www.github.com/OpenA3XX - FLT-CTL (CPT) Panel V1.0"
- board text removed: "10"
- board text removed: "2"
- board text removed: "9"
- board text removed: "https://www.gitgub.com/OpenA3XX - FLT-CTL (CPT) Panel V1.0"
