File: overhead/left/flt-ctl/electronics/fl-ctl/fl-ctl.kicad_sch (KiCad schematic)
At the start: 29 parts, among them J1 Conn_02x01, J2 Conn_02x05_Counter_Clockwise

Commit message: Gerber Files generation and updates
Parts:
- removed J2: Conn_02x05_Counter_Clockwise, Connector_PinHeader_2.54mm:PinHeader_2x05_P2.54mm_Vertical, symbol Connector_Generic:Conn_02x05_Counter_Clockwise
- added J2: Conn_02x20_Counter_Clockwise, Connector_PinHeader_2.54mm:PinHeader_2x20_P2.54mm_Vertical, symbol Connector_Generic:Conn_02x20_Counter_Clockwise
- added J7: Conn_02x01, TerminalBlock:TerminalBlock_bornier-2_P5.08mm, symbol Connector_Generic:Conn_02x01
Connections:
- net +12V: now also J7.2 (Pin_2)
- net GND: now also J7.1 (Pin_1)
- net at KR1.1 (+5V_TOP_LED): now also J2.1 (Pin_1)
- net at KR1.3 (+5V_BOTTOM_LED): now also J2.2 (Pin_2)
- net at KR1.5 (SW_IN): now also J2.3 (Pin_3)
- net at KR2.1 (+5V_TOP_LED): now also J2.4 (Pin_4)
- net at KR2.3 (+5V_BOTTOM_LED): now also J2.5 (Pin_5)
- net at KR2.5 (SW_IN): now also J2.6 (Pin_6)
- net at KR3.1 (+5V_TOP_LED): now also J2.7 (Pin_7)
- net at KR3.3 (+5V_BOTTOM_LED): now also J2.8 (Pin_8)
- net at KR3.5 (SW_IN): now also J2.9 (Pin_9)
- no-connect marks 1 -> 31
