File: overhead/left/oxygen_calls_rain-rplnt_wipers/electronics/oxygen_calls_rain-rplnt_wipers.kicad_pcb (KiCad board)
At the start: 2 copper layers, 145 x 170.2 mm, 75 parts, among them J1 Conn_02x01, J2 Conn_02x11_Counter_Clockwise, J3 Conn_02x01, J4 Conn_02x01, J5 Conn_02x01, J6 Conn_02x01, J7 Conn_02x01, J8 Conn_02x01, J9 Conn_02x02_Counter_Clockwise

Commit message: Updated OCRW PCB Iteration 2
Parts:
- added KR5: ~, OpenA3XX:Korry Switch, F.Cu at (71.5, 41.4)
- J2: value Conn_02x11_Counter_Clockwise -> Conn_02x01; footprint Connector_PinHeader_2.54mm:PinHeader_2x11_P2.54mm_Vertical -> TerminalBlock:TerminalBlock_bornier-2_P5.08mm
- J3: value Conn_02x01 -> Conn_02x20_Counter_Clockwise; footprint Connector_PinHeader_2.54mm:PinHeader_1x02_P2.54mm_Vertical -> Connector_PinHeader_2.54mm:PinHeader_2x20_P2.54mm_Vertical; moved to B.Cu
- moved J2 149.6 mm to (89.2, 26.2)
- moved J1 139.1 mm to (157.0, 26.2), turned to 0 degrees
- moved J3 117.7 mm to (168.0, 126.7), turned to 180 degrees
- moved D12 3.75 mm to (65.2, 53.4)
- moved D15 3.49 mm to (158.9, 35.1)
- moved D2 3.23 mm to (82.3, 30.5)
- moved D6 2.08 mm to (136.6, 33.4)
- moved D5 1.06 mm to (115.4, 31.3)
Connections:
- J2 pad 2: GND -> +12V
- J3 pad 2: Net-(J2-Pin_16) -> GND
- J4 pad 2: Net-(J2-Pin_13) -> Net-(J3-Pin_13)
- J5 pad 2: Net-(J2-Pin_17) -> Net-(J3-Pin_17)
- J6 pad 2: Net-(J2-Pin_14) -> Net-(J3-Pin_14)
- J7 pad 2: Net-(J2-Pin_18) -> Net-(J3-Pin_18)
- J8 pad 2: Net-(J2-Pin_15) -> Net-(J3-Pin_15)
- J9 pad 2: Net-(J2-Pin_19) -> Net-(J3-Pin_19)
- J9 pad 3: Net-(J2-Pin_20) -> Net-(J3-Pin_20)
- J9 pad 4: Net-(J2-Pin_21) -> Net-(J3-Pin_21)
- KR2 pad 1: Net-(J2-Pin_7) -> Net-(J3-Pin_7)
- KR2 pad 3: Net-(J2-Pin_8) -> Net-(J3-Pin_8)
- KR3 pad 1: Net-(J2-Pin_4) -> Net-(J3-Pin_4)
- KR3 pad 3: Net-(J2-Pin_5) -> Net-(J3-Pin_5)
- KR3 pad 5: Net-(J2-Pin_6) -> Net-(J3-Pin_6)
- KR4 pad 1: Net-(J2-Pin_10) -> Net-(J3-Pin_10)
- KR4 pad 3: Net-(J2-Pin_11) -> Net-(J3-Pin_11)
Routing:
- net Net-(J3-Pin_16): track 0.00 -> 175.1 mm, vias 0 -> 1
- net Net-(J2-Pin_16): track 165.8 -> 0.00 mm, vias 1 -> 0
- net Net-(J2-Pin_6): track 163.8 -> 0.00 mm, vias 4 -> 0
- net Net-(J3-Pin_13): track 0.00 -> 163.2 mm, vias 0 -> 1
- net Net-(J2-Pin_13): track 151.9 -> 0.00 mm, vias 1 -> 0
- net Net-(J2-Pin_14): track 146.2 -> 0.00 mm, vias 4 -> 0
- net Net-(J2-Pin_8): track 141.2 -> 0.00 mm, vias 2 -> 0
- net Net-(J3-Pin_17): track 0.00 -> 134.0 mm, vias 0 -> 1
- net Net-(J3-Pin_7): track 0.00 -> 131.7 mm, vias 0 -> 1
- net Net-(J2-Pin_4): track 129.9 -> 0.00 mm
- net Net-(J2-Pin_7): track 129.7 -> 0.00 mm, vias 1 -> 0
- net Net-(J3-Pin_8): track 0.00 -> 119.1 mm, vias 0 -> 2
- net Net-(J3-Pin_14): track 0.00 -> 109.3 mm, vias 0 -> 2
- net Net-(J2-Pin_17): track 107.2 -> 0.00 mm
- net Net-(J2-Pin_5): track 104.2 -> 0.00 mm
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Other:
- board text added: "1"
- board text added: "40"
