File: overhead/left/oxygen_calls_rain-rplnt_wipers/electronics/oxygen_calls_rain-rplnt_wipers.kicad_sch (KiCad schematic)
At the start: 73 parts, among them J1 Conn_02x01, J2 Conn_02x11_Counter_Clockwise, J3 Conn_02x01, J4 Conn_02x01, J5 Conn_02x01, J6 Conn_02x01, J7 Conn_02x01, J8 Conn_02x01, J9 Conn_02x02_Counter_Clockwise

Commit message: Updated OCRW PCB Iteration 2
Parts:
- removed J2: Conn_02x11_Counter_Clockwise, Connector_PinHeader_2.54mm:PinHeader_2x11_P2.54mm_Vertical, symbol Connector_Generic:Conn_02x11_Counter_Clockwise
- removed J3: Conn_02x01, Connector_PinHeader_2.54mm:PinHeader_1x02_P2.54mm_Vertical, symbol Connector_Generic:Conn_02x01
- added J2: Conn_02x01, TerminalBlock:TerminalBlock_bornier-2_P5.08mm, symbol Connector_Generic:Conn_02x01
- added J3: Conn_02x20_Counter_Clockwise, Connector_PinHeader_2.54mm:PinHeader_2x20_P2.54mm_Vertical, symbol Connector_Generic:Conn_02x20_Counter_Clockwise
- added KR5: ~, OpenA3XX:Korry Switch, symbol KorrySwitch:Korry_Switch
Connections:
- net +12V: now also J2.2 (Pin_2)
- net GND: now also J2.1 (Pin_1), J3.1 (Pin_1), J3.12 (Pin_12), J3.2 (Pin_2), J3.3 (Pin_3), J3.9 (Pin_9), KR5.6 (SW_OUT)
- net at J8.2 (Pin_2): now also J3.15 (Pin_15)
- net at KR4.1 (+5V_TOP_LED): now also J3.10 (Pin_10)
- net at KR4.3 (+5V_BOTTOM_LED): now also J3.11 (Pin_11)
- net at J9.2 (Pin_2): now also J3.19 (Pin_19)
- net at J9.3 (Pin_3): now also J3.20 (Pin_20)
- net at J9.4 (Pin_4): now also J3.21 (Pin_21)
- net at J5.2 (Pin_2): now also J3.17 (Pin_17)
- net at J6.2 (Pin_2): now also J3.14 (Pin_14)
- net at KR3.1 (+5V_TOP_LED): now also J3.4 (Pin_4)
- net at KR3.3 (+5V_BOTTOM_LED): now also J3.5 (Pin_5)
- net at KR3.5 (SW_IN): now also J3.6 (Pin_6)
- net at J4.2 (Pin_2): now also J3.13 (Pin_13)
- net at J7.2 (Pin_2): now also J3.18 (Pin_18)
- net at KR2.1 (+5V_TOP_LED): now also J3.7 (Pin_7)
- net at KR2.3 (+5V_BOTTOM_LED): now also J3.8 (Pin_8)
- new net: J3.16 (Pin_16), KR5.5 (SW_IN)
- no-connect marks 0 -> 23
Other:
- note added: "CALLS AFT"
- note added: "CALLS ALL"
- note added: "CALLS FWD"
- note added: "CALLS MECH"
- note added: "CREW SUPPLY"
- note added: "EMER"
- note added: "HIGH ALT LANDING"
- note added: "MASK MAN ON"
- note added: "PASSENGER"
- note added: "RAIN RPLNT"
- note added: "WIPERS"
- note removed: "Flap Mode"
- note removed: "G/S Mode"
- note removed: "GEN 1 Line"
- note removed: "RAT & EMER GEN"
