File: overhead/left/pa-cockpit_door_video/electronics/pa-cockpit_door_video/pa-cockpit_door_video.kicad_pcb (KiCad board)
At the start: 2 copper layers, 145 x 47.3 mm, 30 parts, among them J1 Conn_02x01, J3 Conn_02x03_Counter_Clockwise

Commit message: Iteration 2 - PCBs
Parts:
- added J2: Conn_02x01, TerminalBlock:TerminalBlock_bornier-2_P5.08mm, B.Cu at (89.7, 113.6)
- J3: value Conn_02x03_Counter_Clockwise -> Conn_02x20_Counter_Clockwise; footprint Connector_PinHeader_2.54mm:PinHeader_2x03_P2.54mm_Vertical -> Connector_PinHeader_2.54mm:PinHeader_2x20_P2.54mm_Vertical
- moved D16 40.3 mm to (157.5, 99.7)
- moved J3 0.98 mm to (212.4, 75.5)
Routing:
- net Net-(D16-K): track 16.9 -> 66.9 mm, vias 0 -> 2
- net Net-(J3-Pin_2): track 114.0 -> 96.2 mm
- net Net-(J3-Pin_3): track 129.4 -> 113.8 mm, vias 2 -> 1
- net GND: track 256.5 -> 271.8 mm
- net Net-(D11-K): track 17.4 -> 30.4 mm, vias 0 -> 2
- net Net-(J3-Pin_1): track 101.8 -> 93.8 mm, vias 3 -> 1
- net Net-(D8-K): track 75.8 -> 83.6 mm
- net +12V: track 221.1 -> 216.4 mm, vias 6 -> 5
- net Net-(D17-K): track 17.8 -> 21.7 mm, vias 0 -> 2
- net Net-(D15-K): track 8.76 -> 12.7 mm, vias 0 -> 2
- net Net-(D4-K): track 39.4 -> 42.7 mm, vias 0 -> 2
- net Net-(J3-Pin_4): track 30.1 -> 28.2 mm
- net Net-(D2-K): track 21.2 -> 19.3 mm
- net Net-(D6-K): track 25.0 -> 23.6 mm
- net Net-(J3-Pin_5): track 30.2 -> 29.1 mm
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Other:
- board text added: "40"
- board text added: "https://www.github.com/OpenA3XX - PA & COCKPIT DOOR VIDEO V1.0"
- board text removed: "2"
- board text removed: "5"
- board text removed: "6"
- board text removed: "https://www.gitgub.com/OpenA3XX - PA & COCKPIT DOOR VIDEO V1.0"
