File: overhead/left/pa-cockpit_door_video/electronics/pa-cockpit_door_video/pa-cockpit_door_video.kicad_sch (KiCad schematic)
At the start: 28 parts, among them J1 Conn_02x01, J3 Conn_02x03_Counter_Clockwise

Commit message: Iteration 2 - PCBs
Parts:
- removed J3: Conn_02x03_Counter_Clockwise, Connector_PinHeader_2.54mm:PinHeader_2x03_P2.54mm_Vertical, symbol Connector_Generic:Conn_02x03_Counter_Clockwise
- added J2: Conn_02x01, TerminalBlock:TerminalBlock_bornier-2_P5.08mm, symbol Connector_Generic:Conn_02x01
- added J3: Conn_02x20_Counter_Clockwise, Connector_PinHeader_2.54mm:PinHeader_2x20_P2.54mm_Vertical, symbol Connector_Generic:Conn_02x20_Counter_Clockwise
Connections:
- net +12V: now also J2.2 (Pin_2)
- net GND: now also J2.1 (Pin_1)
- net at KR1.1 (+5V_TOP_LED): now also J3.1 (Pin_1)
- net at KR1.3 (+5V_BOTTOM_LED): now also J3.2 (Pin_2)
- net at KR1.5 (SW_IN): now also J3.3 (Pin_3)
- net at KR2.1 (+5V_TOP_LED): now also J3.4 (Pin_4)
- net at KR2.3 (+5V_BOTTOM_LED): now also J3.5 (Pin_5)
- net at KR2.5 (SW_IN): now also J3.6 (Pin_6)
- no-connect marks 0 -> 34
Other:
- moved on the sheet: KR2
