File: overhead/centre/lights/electronics/lights.kicad_sch (KiCad schematic)
At the start: 186 parts, among them J1 Conn_02x20_Counter_Clockwise, J10 Conn_02x20_Counter_Clockwise, J11 Conn_01x03_Pin, J12 Conn_01x04_Pin, J13 Conn_01x09_Pin, J14 Conn_01x03_Pin, J15 Conn_01x03_Pin, J16 Conn_01x04_Pin, J17 Conn_01x04_Pin, J18 Conn_01x04_Pin, J19 Conn_01x04_Pin, J2 Conn_01x03_Pin, J20 Conn_01x03_Pin, J21 Conn_02x01, J3 Conn_01x03_Pin, J4 Conn_01x03_Pin, J5 Conn_01x03_Pin, J6 Conn_01x04_Pin, J7 Conn_01x04_Pin, J8 Conn_01x04_Pin, J9 Conn_01x04_Pin

Commit message: Updated Lights Panel Iteraion 2 Completed
Parts:
- added J22: Conn_02x01, TerminalBlock:TerminalBlock_bornier-2_P5.08mm, symbol Connector_Generic:Conn_02x01
Connections:
- net +12V: now also J22.2 (Pin_2)
- net GND: now also J22.1 (Pin_1)
- net at J1.24 (Pin_24): now also KR6.5 (SW_IN); no longer KR8.1 (+5V_TOP_LED)
- net at J1.25 (Pin_25): now also KR8.1 (+5V_TOP_LED); no longer KR6.5 (SW_IN)
- no-connect marks 0 -> 6
Changed lines of the file:
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@@
 	)
 	(junction
+		(at 535.94 57.15)
+		(diameter 0)
+		(color 0 0 0 0)
+	)
+	(junction
 		(at 106.68 187.96)
 		(diameter 0)
@@
 		(color 0 0 0 0)
 	)
+	(no_connect
+		(at 396.24 62.23)
+	)
+	(no_connect
+		(at 173.99 29.21)
+	)
+	(no_connect
+		(at 173.99 26.67)
+	)
+	(no_connect
+		(at 396.24 59.69)
+	)
+	(no_connect
+		(at 396.24 54.61)
+	)
+	(no_connect
+		(at 396.24 57.15)
+	)
 	(wire
 		(pts
@@
 	(wire
 		(pts
-			(xy 182.88 64.77) (xy 173.99 64.77)
-		)
-		(stroke
-			(width 0)
-			(type default)
-		)
-	)
-	(wire
-		(pts
 			(xy 228.6 316.23) (xy 228.6 311.15)
 		)
@@
 	(wire
 		(pts
+			(xy 173.99 67.31) (xy 182.88 67.31)
+		)
+		(stroke
+			(width 0)
+			(type default)
+		)
+	)
+	(wire
+		(pts
 			(xy 427.99 60.96) (xy 427.99 111.76)
 		)
@@
 	(wire
 		(pts
+			(xy 525.78 43.18) (xy 525.78 41.91)
+		)
+		(stroke
+			(width 0)
+			(type default)
+		)
+	)
+	(wire
+		(pts
 			(xy 91.44 165.1) (xy 59.69 165.1)
 		)
@@
 	(wire
 		(pts
-			(xy 535.94 55.88) (xy 535.94 59.69)
+			(xy 535.94 55.88) (xy 535.94 57.15)
 		)
 		(stroke
@@
 	(wire
 		(pts
+			(xy 173.99 64.77) (xy 181.61 64.77)
+		)
+		(stroke
+			(width 0)
+			(type default)
+		)
+	)
+	(wire
+		(pts
 			(xy 360.68 443.23) (xy 370.84 443.23)
 		)
@@
 	(wire
 		(pts
-			(xy 181.61 85.09) (xy 181.61 67.31)
+			(xy 181.61 64.77) (xy 181.61 85.09)
 		)
 		(stroke
@@
 	(wire
 		(pts
-			(xy 182.88 87.63) (xy 182.88 64.77)
+			(xy 182.88 87.63) (xy 182.88 67.31)
 		)
 		(stroke
@@
 	(wire
 		(pts
+			(xy 525.78 55.88) (xy 525.78 57.15)
+		)
+		(stroke
+			(width 0)
+			(type default)
+		)
+	)
+	(wire
+		(pts
 			(xy 170.18 449.58) (xy 193.04 449.58)
 		)
@@
 	(wire
 		(pts
+			(xy 535.94 57.15) (xy 535.94 59.69)
+		)
+		(stroke
+			(width 0)
+			(type default)
+		)
+	)
+	(wire
+		(pts
 			(xy 293.37 33.02) (xy 317.5 33.02)
 		)
@@
 	(wire
 		(pts
-			(xy 181.61 67.31) (xy 173.99 67.31)
-		)
-		(stroke
-			(width 0)
-			(type default)
-		)
-	)
-	(wire
-		(pts
 			(xy 359.41 59.69) (xy 383.54 59.69)
 		)
@@
 	(wire
 		(pts
+			(xy 525.78 57.15) (xy 535.94 57.15)
+		)
+		(stroke
+			(width 0)
+			(type default)
+		)
+	)
+	(wire
+		(pts
 			(xy 137.16 326.39) (xy 148.59 326.39)
 		)
@@
 	(wire
 		(pts
+			(xy 525.78 41.91) (xy 535.94 41.91)
+		)
+		(stroke
+			(width 0)
+			(type default)
+		)
+	)
+	(wire
+		(pts
 			(xy 120.65 54.61) (xy 161.29 54.61)
 		)
@@
 		)
 		(property "Description" "MAN VS CTL"
-			(at 477.52 25.146 0)
+			(at 489.712 30.734 0)
 			(effects
 				(font
@@
 		)
 		(property "Description" "Seat Belts"
-			(at 476.25 107.95 0)
+			(at 483.616 113.538 0)
 			(effects
 				(font
@@
 		(on_board yes)
 		(dnp no)
-		(fields_autoplaced yes)
 		(property "Reference" "J5"
 			(at 321.945 86.36 0)
@@
 		)
 		(property "Description" "RWY Turn Off"
-			(at 322.58 78.74 0)
+			(at 330.454 78.74 0)
 			(effects
 				(font
@@
 		(on_board yes)
 		(dnp no)
-		(fields_autoplaced yes)
 		(property "Reference" "J6"
 			(at 323.85 99.0599 0)
@@
 		)
 		(property "Description" "Land L"
-			(at 322.58 101.6 0)
+			(at 330.2 99.06 0)
 			(effects
 				(font
@@
 		(on_board yes)
 		(dnp no)
-		(fields_autoplaced yes)
 		(property "Reference" "J2"
 			(at 321.945 40.64 0)
@@
 		)
 		(property "Description" "Strobe"
-			(at 322.58 33.02 0)
+			(at 327.914 33.274 0)
 			(effects
 				(font
@@
 		)
 		(property "Description" "OVHD LIGHTS"
-			(at 481.584 76.708 0)
+			(at 501.396 83.82 0)
 			(effects
 				(font
@@
 		)
 		(property "Description" "ICE IND & STBY COMPASS"
-			(at 478.028 100.584 0)
+			(at 491.49 95.504 0)
 			(effects
 				(font
@@
 		)
 		(property "Description" "Land R"
-			(at 323.596 110.998 0)
+			(at 330.454 113.03 0)
 			(effects
 				(font
@@
 		(on_board yes)
 		(dnp no)
-		(fields_autoplaced yes)
 		(property "Reference" "J9"
 			(at 323.85 147.3199 0)
@@
 		)
 		(property "Description" "Nose"
-			(at 322.58 149.86 0)
+			(at 329.438 147.574 0)
 			(effects
 				(font
@@
 		)
 		(property "Description" "Dome Light"
-			(at 480.314 124.714 0)
+			(at 488.442 128.27 0)
 			(effects
 				(font
@@
 	)
 	(symbol
+		(lib_id "Connector_Generic:Conn_02x01")
+		(at 525.78 50.8 90)
+		(unit 1)
+		(exclude_from_sim no)
+		(in_bom yes)
+		(on_board yes)
+		(dnp no)
+		(property "Reference" "J22"
+			(at 520.2682 49.53 0)
+			(effects
+				(font
+					(size 1.27 1.27)
+				)
+			)
+		)
+		(property "Value" "Conn_02x01"
+			(at 522.5796 49.53 0)
+			(effects
+				(font
+					(size 1.27 1.27)
+				)
+			)
+		)
+		(property "Footprint" "TerminalBlock:TerminalBlock_bornier-2_P5.08mm"
+			(at 525.78 50.8 0)
+			(effects
+				(font
+					(size 1.27 1.27)
+				)
+				(hide yes)
+			)
+		)
+		(property "Datasheet" "~"
+			(at 525.78 50.8 0)
+			(effects
+				(font
+					(size 1.27 1.27)
+				)
+				(hide yes)
+			)
+		)
+		(property "Description" "Generic connector, double row, 02x01, this symbol is compatible with counter-clockwise, top-bottom and odd-even numbering schemes., script generated (kicad-library-utils/schlib/autogen/connector/)"
+			(at 469.9 44.45 0)
+			(effects
+				(font
+					(size 1.27 1.27)
+				)
+				(hide yes)
+			)
+		)
+		(pin "1"
+		)
+		(pin "2"
+		)
+		(instances
+			(project "lights"
+				(path "/53f067b2-5e62-40c9-af08-fed5b43764dd"
+					(reference "J22")
+					(unit 1)
+				)
+			)
+		)
+	)
+	(symbol
 		(lib_id "power:GND")
 		(at 270.51 457.2 0)
@@
 		(on_board yes)
 		(dnp no)
-		(fields_autoplaced yes)
 		(property "Reference" "J3"
 			(at 321.945 55.88 0)
@@
 		)
 		(property "Description" "Beacon"
-			(at 322.58 48.26 0)
+			(at 327.406 48.514 0)
 			(effects
 				(font
@@
 		)
 		(property "Description" "No Smoking"
-			(at 480.822 155.194 0)
+			(at 488.696 158.75 0)
 			(effects
 				(font
@@
 		)
 		(property "Description" "Ember Exit LT"
-			(at 482.092 171.45 0)
+			(at 489.712 175.26 0)
 			(effects
 				(font
@@
 		(on_board yes)
 		(dnp no)
-		(fields_autoplaced yes)
 		(property "Reference" "J4"
 			(at 321.945 71.12 0)
@@
 		)
 		(property "Description" "Wing"
-			(at 322.58 63.5 0)
+			(at 326.644 63.5 0)
 			(effects
 				(font
@@
 		)
 		(property "Description" "ANN LT"
-			(at 478.79 139.7 0)
+			(at 486.41 143.51 0)
 			(effects
 				(font
@@
 		(on_board yes)
 		(dnp no)
-		(fields_autoplaced yes)
 		(property "Reference" "J8"
 			(at 323.85 128.2699 0)
@@
 		)
 		(property "Description" "Nav & Logo"
-			(at 322.58 130.81 0)
+			(at 332.486 128.524 0)
 			(effects
 				(font
@@
 		)
 		(property "Description" "LDG ELEV"
-			(at 476.504 42.926 0)
+			(at 483.362 55.88 0)
 			(effects
 				(font
