File: overhead/centre/aircond/electronics/aircond/aircond.kicad_pcb (KiCad board)
At the start: 2 copper layers, 322.4 x 112.7 mm, 181 parts, among them J1 Conn_02x20_Counter_Clockwise, J2 Conn_01x09_Pin, J3 Conn_01x09_Pin, J4 Conn_01x09_Pin, J5 Conn_01x04_Pin, J6 Conn_01x04_Pin, J7 Conn_02x20_Counter_Clockwise, J8 Conn_02x01

Commit message: Iteration2 AIRCOND Panel
Parts:
- added J9: Conn_02x01, TerminalBlock:TerminalBlock_bornier-2_P5.08mm, B.Cu at (71.8, 191.5)
Routing:
- net Net-(D53-K): track 20.7 -> 78.8 mm, vias 0 -> 2
- net Net-(D48-K): track 22.8 -> 44.9 mm
- net GND: track 1346.0 -> 1325.7 mm, vias 19 -> 16
- net +12V: track 1200.0 -> 1215.1 mm, vias 27 -> 23
- net Net-(D117-K): track 29.4 -> 44.1 mm, vias 0 -> 2
- net Net-(J1-Pin_3): track 117.7 -> 131.8 mm
- net Net-(J6-Pin_1): track 137.4 -> 149.9 mm
- net Net-(D78-K): track 28.7 -> 16.4 mm, vias 2 -> 0
- net Net-(J1-Pin_1): track 100.3 -> 112.4 mm
- net Net-(J4-Pin_3): track 108.9 -> 96.8 mm
- net Net-(J1-Pin_32): track 134.7 -> 146.5 mm
- net Net-(J1-Pin_7): track 274.8 -> 265.3 mm
- net Net-(D68-K): track 11.6 -> 21.1 mm, vias 0 -> 2
- net Net-(D62-K): track 23.7 -> 14.5 mm
- net Net-(J5-Pin_3): track 248.6 -> 257.7 mm, vias 2 -> 3
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Other:
- board size 322.4 x 112.7 mm -> 322.4 x 113.3 mm
- board text added: "+12V Variable Backlight"
- board text added: "1"
- board text added: "40"
- board text added: "GND"
- board text added: "[CONNECTION J1] 1-PACK-1-TOP_LED 2-PACK-1-BOTTOM_LED 3-PACK-1-KORRY_SW 4-PACK-2-TOP_LED 5-PACK-2-BOTTOM_LED 6-PACK-2-KORRY_SW 7-ENGINE-2-BLEED-TOP_LED 8-ENGINE-2-BLEED-BOTTOM_LED 9-ENGINE-2-BLEED-KORRY_SW 10-HOT-AIR-TOP_LED 11-HOT-AIR-BOTTOM_LED 12-HOT-AIR-KORRY_SW 13-APU-BLEED-TOP_LED 14-APU-BLEED-BOTTOM_LED 15-APU-BLEED-KORRY_SW 16-ENGINE-1-BLEED-TOP_LED 17-ENGINE-1-BLEED-BOTTOM_LED 18-ENGINE-1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"
- board text added: "[CONNECTION J7] 1-PACKS-AFT_CABIN-POS1-SW 2-PACKS-AFT_CABIN-POS2-SW 3-PACKS-AFT_CABIN-POS3-SW 4-PACKS-AFT_CABIN-POS4-SW 5-PACKS-AFT_CABIN-POS5-SW 6-PACKS-AFT_CABIN-POS6-SW 7-PACKS-AFT_CABIN-POS7-SW 8-PACKS-AFT_CABIN-POS8-SW 9-PACKS-FLOW-POS1-SW 10-PACKS-FLOW-POS2-SW 11-PACKS-FLOW-POS3-SW 12-X-BLEED-POS1-SW 13-X-BLEED-POS2-SW 14-X-BLEED-POS3-SW"
