File: overhead/centre/aircond/electronics/aircond/aircond.kicad_sch (KiCad schematic)
At the start: 179 parts, among them J1 Conn_02x20_Counter_Clockwise, J2 Conn_01x09_Pin, J3 Conn_01x09_Pin, J4 Conn_01x09_Pin, J5 Conn_01x04_Pin, J6 Conn_01x04_Pin, J7 Conn_02x20_Counter_Clockwise, J8 Conn_02x01

Commit message: Iteration2 AIRCOND Panel
Parts:
- added J9: Conn_02x01, TerminalBlock:TerminalBlock_bornier-2_P5.08mm, symbol Connector_Generic:Conn_02x01
Connections:
- net +12V: now also J9.2 (Pin_2)
- net GND: now also J9.1 (Pin_1)
Changed lines of the file:
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@@
 	)
 	(junction
+		(at 372.11 49.53)
+		(diameter 0)
+		(color 0 0 0 0)
+	)
+	(junction
 		(at 270.51 64.77)
 		(diameter 0)
@@
 	(wire
 		(pts
+			(xy 360.68 35.56) (xy 360.68 34.29)
+		)
+		(stroke
+			(width 0)
+			(type default)
+		)
+	)
+	(wire
+		(pts
 			(xy 95.25 173.99) (xy 80.01 173.99)
 		)
@@
 	(wire
 		(pts
+			(xy 360.68 34.29) (xy 372.11 34.29)
+		)
+		(stroke
+			(width 0)
+			(type default)
+		)
+	)
+	(wire
+		(pts
 			(xy 167.64 236.22) (xy 190.5 236.22)
 		)
@@
 	(wire
 		(pts
+			(xy 360.68 49.53) (xy 372.11 49.53)
+		)
+		(stroke
+			(width 0)
+			(type default)
+		)
+	)
+	(wire
+		(pts
 			(xy 99.06 374.65) (xy 106.68 374.65)
 		)
@@
 	(wire
 		(pts
-			(xy 372.11 48.26) (xy 372.11 52.07)
+			(xy 372.11 48.26) (xy 372.11 49.53)
 		)
 		(stroke
@@
 	(wire
 		(pts
+			(xy 360.68 48.26) (xy 360.68 49.53)
+		)
+		(stroke
+			(width 0)
+			(type default)
+		)
+	)
+	(wire
+		(pts
 			(xy 156.21 421.64) (xy 156.21 424.18)
 		)
@@
 	(wire
 		(pts
+			(xy 372.11 49.53) (xy 372.11 52.07)
+		)
+		(stroke
+			(width 0)
+			(type default)
+		)
+	)
+	(wire
+		(pts
 			(xy 72.39 331.47) (xy 62.23 331.47)
 		)
@@
 			)
 		)
-		(property "Description" "MAN VS CTL"
+		(property "Description" "XBLEED"
 			(at 257.81 84.074 0)
 			(effects
@@
 	)
 	(symbol
+		(lib_id "Connector_Generic:Conn_02x01")
+		(at 360.68 43.18 90)
+		(unit 1)
+		(exclude_from_sim no)
+		(in_bom yes)
+		(on_board yes)
+		(dnp no)
+		(property "Reference" "J9"
+			(at 355.1682 41.91 0)
+			(effects
+				(font
+					(size 1.27 1.27)
+				)
+			)
+		)
+		(property "Value" "Conn_02x01"
+			(at 357.4796 41.91 0)
+			(effects
+				(font
+					(size 1.27 1.27)
+				)
+			)
+		)
+		(property "Footprint" "TerminalBlock:TerminalBlock_bornier-2_P5.08mm"
+			(at 360.68 43.18 0)
+			(effects
+				(font
+					(size 1.27 1.27)
+				)
+				(hide yes)
+			)
+		)
+		(property "Datasheet" "~"
+			(at 360.68 43.18 0)
+			(effects
+				(font
+					(size 1.27 1.27)
+				)
+				(hide yes)
+			)
+		)
+		(property "Description" "Generic connector, double row, 02x01, this symbol is compatible with counter-clockwise, top-bottom and odd-even numbering schemes., script generated (kicad-library-utils/schlib/autogen/connector/)"
+			(at 304.8 36.83 0)
+			(effects
+				(font
+					(size 1.27 1.27)
+				)
+				(hide yes)
+			)
+		)
+		(pin "1"
+		)
+		(pin "2"
+		)
+		(instances
+			(project "aircond"
+				(path "/1a545166-1e6c-40d5-a989-dd86e2adc0d0"
+					(reference "J9")
+					(unit 1)
+				)
+			)
+		)
+	)
+	(symbol
 		(lib_id "power:GND")
 		(at 156.21 424.18 0)
@@
 		(on_board yes)
 		(dnp no)
-		(fields_autoplaced yes)
 		(property "Reference" "KR4"
-			(at 116.84 179.7049 0)
+			(at 116.84 178.4349 0)
 			(effects
 				(font
@@
 		)
 		(property "Value" "~"
-			(at 116.84 181.61 0)
+			(at 116.84 180.34 0)
 			(effects
 				(font
@@
 			)
 		)
-		(property "Description" "APU Master SW"
-			(at 105.41 171.45 0)
+		(property "Description" "RAM AIR"
+			(at 102.87 170.942 0)
 			(effects
 				(font
 					(size 1.27 1.27)
 				)
+				(justify left)
 			)
 		)
@@
 			)
 		)
-		(property "Description" "LDG ELEV"
+		(property "Description" "PACKS FWD CABIN"
 			(at 198.374 30.226 0)
 			(effects
@@
 		(on_board yes)
 		(dnp no)
-		(fields_autoplaced yes)
 		(property "Reference" "KR7"
-			(at 252.73 141.6049 0)
+			(at 252.73 140.3349 0)
 			(effects
 				(font
@@
 		)
 		(property "Value" "~"
-			(at 252.73 143.51 0)
+			(at 252.73 142.24 0)
 			(effects
 				(font
@@
 			)
 		)
-		(property "Description" "Cabin Press Mode Sel"
-			(at 241.3 133.35 0)
+		(property "Description" "APU BLEED"
+			(at 236.982 133.096 0)
 			(effects
 				(font
 					(size 1.27 1.27)
 				)
+				(justify left)
 			)
 		)
@@
 		(on_board yes)
 		(dnp no)
-		(fields_autoplaced yes)
 		(property "Reference" "KR6"
-			(at 203.2 140.3349 0)
+			(at 203.2 139.0649 0)
 			(effects
 				(font
@@
 		)
 		(property "Value" "~"
-			(at 203.2 142.24 0)
+			(at 203.2 140.97 0)
 			(effects
 				(font
@@
 			)
 		)
-		(property "Description" "Probe Window Heat"
-			(at 191.77 132.08 0)
+		(property "Description" "HOT AIR"
+			(at 188.722 132.08 0)
 			(effects
 				(font
 					(size 1.27 1.27)
 				)
+				(justify left)
 			)
 		)
@@
 		(on_board yes)
 		(dnp no)
-		(fields_autoplaced yes)
 		(property "Reference" "KR3"
-			(at 115.57 140.3349 0)
+			(at 115.57 139.0649 0)
 			(effects
 				(font
@@
 		)
 		(property "Value" "~"
-			(at 115.57 142.24 0)
+			(at 115.57 140.97 0)
 			(effects
 				(font
@@
 			)
 		)
-		(property "Description" "Anti-Ice Eng 1"
-			(at 104.14 132.08 0)
+		(property "Description" "PACK 2"
+			(at 100.838 131.826 0)
 			(effects
 				(font
 					(size 1.27 1.27)
 				)
+				(justify left)
 			)
 		)
@@
 			)
 		)
-		(property "Description" "LDG ELEV"
-			(at 258.826 52.324 0)
+		(property "Description" "PACKS AFT CABIN"
+			(at 249.174 39.624 0)
 			(effects
 				(font
@@
 			)
 		)
-		(property "Description" "MAN VS CTL"
-			(at 257.81 67.564 0)
+		(property "Description" "PACK FLOW"
+			(at 248.158 62.484 0)
 			(effects
 				(font
@@
 			)
 		)
-		(property "Description" "Anti-Ice Wing"
+		(property "Description" "PACK 1"
 			(at 56.388 131.318 0)
 			(effects
@@
 		(on_board yes)
 		(dnp no)
-		(fields_autoplaced yes)
 		(property "Reference" "KR2"
-			(at 72.39 179.7049 0)
+			(at 72.39 178.4349 0)
 			(effects
 				(font
@@
 		)
 		(property "Value" "~"
-			(at 72.39 181.61 0)
+			(at 72.39 180.34 0)
 			(effects
 				(font
@@
 			)
 		)
-		(property "Description" "Ditching"
-			(at 60.96 171.45 0)
+		(property "Description" "ENGINE 1 BLEED"
+			(at 53.34 170.942 0)
 			(effects
 				(font
 					(size 1.27 1.27)
 				)
+				(justify left)
 			)
 		)
@@
 		(on_board yes)
 		(dnp no)
-		(fields_autoplaced yes)
 		(property "Reference" "KR5"
-			(at 162.56 140.3349 0)
+			(at 162.56 139.0649 0)
 			(effects
 				(font
@@
 		)
 		(property "Value" "~"
-			(at 162.56 142.24 0)
+			(at 162.56 140.97 0)
 			(effects
 				(font
@@
 			)
 		)
-		(property "Description" "Anti-Ice Eng 2"
-			(at 151.13 132.08 0)
+		(property "Description" "ENGINE 2 BLEED"
+			(at 144.272 131.826 0)
 			(effects
 				(font
 					(size 1.27 1.27)
 				)
+				(justify left)
 			)
 		)
@@
 			)
 		)
-		(property "Description" "LDG ELEV"
-			(at 186.944 50.546 0)
+		(property "Description" "PACKS COCKPIT"
+			(at 187.198 80.01 0)
 			(effects
 				(font
