File: overhead/centre/elec/electronics/elec.kicad_pcb (KiCad board)
At the start: 2 copper layers, 322.3 x 106.5 mm, 137 parts, among them IC1 MAX7219CWG, J1 Conn_02x01, J2 Conn_02x20_Counter_Clockwise, P1 Conn_01x02, P2 DataIn

Commit message: Updated Panels ELEC
Parts:
- added J3: Conn_02x01, TerminalBlock:TerminalBlock_bornier-2_P5.08mm, B.Cu at (67.6, 197.4)
- moved D1 2.35 mm to (346.6, 109.0)
Routing:
- net +12V: track 922.5 -> 1063.4 mm, vias 22 -> 21
- net Net-(J2-Pin_1): track 244.2 -> 282.9 mm, vias 0 -> 2
- net Net-(J2-Pin_20): track 259.9 -> 295.8 mm, vias 1 -> 2
- net Net-(D63-K): track 15.3 -> 49.4 mm, vias 2 -> 0
- net Net-(D61-K): track 14.7 -> 40.0 mm, vias 0 -> 2
- net Net-(J2-Pin_11): track 139.9 -> 118.6 mm
- net Net-(J2-Pin_33): track 142.4 -> 125.5 mm, vias 2 -> 1
- net Net-(D43-K): track 30.1 -> 43.7 mm
- net /A_SegA: track 142.7 -> 129.9 mm, vias 4 -> 1
- net Net-(D39-K): track 25.5 -> 35.9 mm, vias 0 -> 2
- net Net-(D38-K): track 10.2 -> 20.1 mm, vias 0 -> 2
- net /A3: track 82.8 -> 92.6 mm
- net Net-(J2-Pin_25): track 153.8 -> 144.1 mm, vias 1 -> 2
- net Net-(D47-K): track 26.0 -> 35.4 mm
- net Net-(J2-Pin_17): track 259.9 -> 267.6 mm
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Other:
- board text added: "+12V Variable Backlight"
- board text added: "+5V (7SEGMENT DRIVER)"
- board text added: "1"
- board text added: "40"
- board text added: "CLK"
- board text added: "DIN"
- board text added: "GND"
- board text added: "MAX7219CWG"
- board text added: "SEL"

Commit message: Changes
Changes
Other:
- board text added: "[CONNECTION J2] 1-COMMERCIAL-TOP_LED 2-COMMERCIAL-BOTTOM_LED 3-COMMERCIAL-KORRY_SW 4-IDG-1-TOP_LED 5-IDG-1-BOTTOM_LED 6-IDG-1-KORRY_SW 7-APU-GEN-TOP_LED 8-APU-GEN-BOTTOM_LED 9-APU-GEN-KORRY_SW 10-EXT-PWR-TOP_LED 11-EXT-PWR-BOTTOM_LED 12-EXT-PWR-KORRY_SW 13-GEN-2-TOP_LED 14-GEN-2-BOTTOM_LED 15-GEN-2-KORRY_SW 16-GALY-CAB-TOP_LED 17-GALY-CAB-BOTTOM_LED 18-GALY-CAB-KORRY_SW 19-GEN-1-TOP_LED 20-GEN-1-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"
Changed lines of the file:
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@@
+		)
+	)
+	(gr_text "[CONNECTION J2]\n1-COMMERCIAL-TOP_LED\n2-COMMERCIAL-BOTTOM_LED\n3-COMMERCIAL-KORRY_SW\n4-IDG-1-TOP_LED\n5-IDG-1-BOTTOM_LED\n6-IDG-1-KORRY_SW\n7-APU-GEN-TOP_LED\n8-APU-GEN-BOTTOM_LED\n9-APU-GEN-KORRY_SW\n10-EXT-PWR-TOP_LED\n11-EXT-PWR-BOTTOM_LED\n12-EXT-PWR-KORRY_SW\n13-GEN-2-TOP_LED\n14-GEN-2-BOTTOM_LED\n15-GEN-2-KORRY_SW\n16-GALY-CAB-TOP_LED\n17-GALY-CAB-BOTTOM_LED\n18-GALY-CAB-KORRY_SW\n19-GEN-1-TOP_LED\n20-GEN-1-BOTTOM_LED\n21-GEN-1-KORRY_SW\n22-BUS-TIE-TOP_LED\n23-BUS-TIE-BOTTOM_LED\n24-BUS-TIE-KORRY_SW\n25-AC-ESS-BUS-TOP_LED\n26-AC-ESS-BUS-BOTTOM_LED\n27-AC-ESS-BUS-KORRY_SW\n28-IDG-2-TOP_LED\n29-IDG-2-BOTTOM_LED\n30-IDG-2-KORRY_SW\n31-BAT-1-TOP_LED\n32-BAT-1-BOTTOM_LED\n33-BAT-1-KORRY_SW\n34-BAT-2-TOP_LED\n35-BAT-2-BOTTOM_LED\n36-BAT-2-KORRY_SW"
+		(at 351.6 158.65 -0)
+		(layer "B.SilkS")
+		(effects
+			(font
+				(size 0.5 0.5)
+				(thickness 0.125)
+				(bold yes)
+			)
+			(justify left bottom mirror)
 		)
 	)
