File: overhead/centre/hyd-fuel/electronics/hyd-fuel.kicad_pcb (KiCad board)
At the start: 2 copper layers, 322.3 x 133.3 mm, 146 parts, among them J1 Conn_02x20_Counter_Clockwise, J2 Conn_01x03_Pin, J3 Conn_02x01

Commit message: Changes
Changes
Parts:
- removed J2: Conn_01x03_Pin, Connector_PinHeader_2.54mm:PinHeader_1x03_P2.54mm_Vertical
- added J4: Conn_02x01, TerminalBlock:TerminalBlock_bornier-2_P5.08mm, B.Cu at (72.0, 208.7)
- added J5: Conn_02x20_Counter_Clockwise, Connector_PinHeader_2.54mm:PinHeader_2x20_P2.54mm_Vertical, B.Cu at (184.8, 86.3)
- added KR14: ~, OpenA3XX:Korry Switch, F.Cu at (149.1, 114.8)
Connections:
- J1 pad 10: Net-(J1-Pin_10) -> unconnected-(J1-Pin_10-Pad10)
- J1 pad 11: Net-(J1-Pin_11) -> unconnected-(J1-Pin_11-Pad11)
- J1 pad 12: Net-(J1-Pin_12) -> unconnected-(J1-Pin_12-Pad12)
- J1 pad 13: Net-(J1-Pin_13) -> unconnected-(J1-Pin_13-Pad13)
- J1 pad 14: Net-(J1-Pin_14) -> unconnected-(J1-Pin_14-Pad14)
- J1 pad 15: Net-(J1-Pin_15) -> unconnected-(J1-Pin_15-Pad15)
- J1 pad 16: Net-(J1-Pin_16) -> unconnected-(J1-Pin_16-Pad16)
- J1 pad 17: Net-(J1-Pin_17) -> unconnected-(J1-Pin_17-Pad17)
- J1 pad 18: Net-(J1-Pin_18) -> unconnected-(J1-Pin_18-Pad18)
- J1 pad 19: Net-(J1-Pin_19) -> unconnected-(J1-Pin_19-Pad19)
- J1 pad 20: Net-(J1-Pin_20) -> unconnected-(J1-Pin_20-Pad20)
- J1 pad 21: Net-(J1-Pin_21) -> unconnected-(J1-Pin_21-Pad21)
- J1 pad 22: Net-(J1-Pin_22) -> unconnected-(J1-Pin_22-Pad22)
- J1 pad 23: Net-(J1-Pin_23) -> unconnected-(J1-Pin_23-Pad23)
- J1 pad 24: Net-(J1-Pin_24) -> unconnected-(J1-Pin_24-Pad24)
- J1 pad 25: Net-(J1-Pin_25) -> unconnected-(J1-Pin_25-Pad25)
- J1 pad 26: Net-(J1-Pin_26) -> unconnected-(J1-Pin_26-Pad26)
- J1 pad 27: Net-(J1-Pin_27) -> unconnected-(J1-Pin_27-Pad27)
- J1 pad 28: Net-(J1-Pin_28) -> unconnected-(J1-Pin_28-Pad28)
- J1 pad 29: Net-(J1-Pin_29) -> unconnected-(J1-Pin_29-Pad29)
- J1 pad 30: Net-(J1-Pin_30) -> unconnected-(J1-Pin_30-Pad30)
- J1 pad 31: Net-(J1-Pin_31) -> unconnected-(J1-Pin_31-Pad31)
- J1 pad 32: Net-(J1-Pin_32) -> unconnected-(J1-Pin_32-Pad32)
- J1 pad 33: Net-(J1-Pin_33) -> unconnected-(J1-Pin_33-Pad33)
- J1 pad 34: Net-(J1-Pin_34) -> unconnected-(J1-Pin_34-Pad34)
- J1 pad 35: Net-(J1-Pin_35) -> unconnected-(J1-Pin_35-Pad35)
- J1 pad 36: Net-(J1-Pin_36) -> unconnected-(J1-Pin_36-Pad36)
- J1 pad 37: Net-(J1-Pin_37) -> unconnected-(J1-Pin_37-Pad37)
- J1 pad 38: Net-(J1-Pin_38) -> unconnected-(J1-Pin_38-Pad38)
- J1 pad 39: Net-(J1-Pin_39) -> unconnected-(J1-Pin_39-Pad39)
- J1 pad 4: Net-(J1-Pin_4) -> unconnected-(J1-Pin_4-Pad4)
- J1 pad 40: Net-(J1-Pin_40) -> unconnected-(J1-Pin_40-Pad40)
- J1 pad 5: Net-(J1-Pin_5) -> unconnected-(J1-Pin_5-Pad5)
- J1 pad 6: Net-(J1-Pin_6) -> unconnected-(J1-Pin_6-Pad6)
- J1 pad 7: Net-(J1-Pin_7) -> unconnected-(J1-Pin_7-Pad7)
- J1 pad 8: Net-(J1-Pin_8) -> unconnected-(J1-Pin_8-Pad8)
- J1 pad 9: Net-(J1-Pin_9) -> unconnected-(J1-Pin_9-Pad9)
- KR1 pad 1: Net-(J1-Pin_1) -> Net-(J5-Pin_1)
- KR1 pad 3: Net-(J1-Pin_2) -> Net-(J5-Pin_2)
- KR1 pad 5: Net-(J1-Pin_3) -> Net-(J5-Pin_3)
- KR10 pad 1: Net-(J1-Pin_34) -> Net-(J5-Pin_34)
- KR10 pad 3: Net-(J1-Pin_35) -> Net-(J5-Pin_35)
- KR10 pad 5: Net-(J1-Pin_36) -> Net-(J5-Pin_36)
- KR11 pad 1: Net-(J1-Pin_16) -> Net-(J5-Pin_16)
- KR11 pad 3: Net-(J1-Pin_17) -> Net-(J5-Pin_17)
- KR11 pad 5: Net-(J1-Pin_18) -> Net-(J5-Pin_18)
- KR12 pad 1: Net-(J1-Pin_37) -> Net-(J5-Pin_37)
- KR12 pad 3: Net-(J1-Pin_38) -> Net-(J5-Pin_38)
- KR12 pad 5: Net-(J1-Pin_39) -> Net-(J5-Pin_39)
- KR13 pad 1: Net-(J1-Pin_19) -> Net-(J5-Pin_19)
- KR13 pad 3: Net-(J1-Pin_20) -> Net-(J5-Pin_20)
- KR13 pad 5: Net-(J1-Pin_21) -> Net-(J5-Pin_21)
- KR2 pad 1: Net-(J1-Pin_22) -> Net-(J5-Pin_22)
- KR2 pad 3: Net-(J1-Pin_23) -> Net-(J5-Pin_23)
- KR2 pad 5: Net-(J1-Pin_24) -> Net-(J5-Pin_24)
- KR3 pad 1: Net-(J1-Pin_4) -> Net-(J5-Pin_4)
- KR3 pad 3: Net-(J1-Pin_5) -> Net-(J5-Pin_5)
- KR3 pad 5: Net-(J1-Pin_6) -> Net-(J5-Pin_6)
- KR4 pad 1: Net-(J1-Pin_25) -> Net-(J5-Pin_25)
- KR4 pad 3: Net-(J1-Pin_26) -> Net-(J5-Pin_26)
- KR4 pad 5: Net-(J1-Pin_27) -> Net-(J5-Pin_27)
- KR5 pad 1: Net-(J1-Pin_7) -> Net-(J5-Pin_7)
- KR5 pad 3: Net-(J1-Pin_8) -> Net-(J5-Pin_8)
- KR5 pad 5: Net-(J1-Pin_9) -> Net-(J5-Pin_9)
- KR6 pad 1: Net-(J1-Pin_28) -> Net-(J5-Pin_28)
- KR6 pad 3: Net-(J1-Pin_29) -> Net-(J5-Pin_29)
- KR6 pad 5: Net-(J1-Pin_30) -> Net-(J5-Pin_30)
- KR7 pad 1: Net-(J1-Pin_10) -> Net-(J5-Pin_10)
- KR7 pad 3: Net-(J1-Pin_11) -> Net-(J5-Pin_11)
- KR7 pad 5: Net-(J1-Pin_12) -> Net-(J5-Pin_12)
- KR8 pad 1: Net-(J1-Pin_31) -> Net-(J5-Pin_31)
- KR8 pad 3: Net-(J1-Pin_32) -> Net-(J5-Pin_32)
- KR8 pad 5: Net-(J1-Pin_33) -> Net-(J5-Pin_33)
- KR9 pad 1: Net-(J1-Pin_13) -> Net-(J5-Pin_13)
- KR9 pad 3: Net-(J1-Pin_14) -> Net-(J5-Pin_14)
- KR9 pad 5: Net-(J1-Pin_15) -> Net-(J5-Pin_15)
Routing:
- net Net-(J5-Pin_38): track 0.00 -> 302.9 mm, vias 0 -> 1
- net Net-(J5-Pin_37): track 0.00 -> 286.9 mm, vias 0 -> 2
- net Net-(J5-Pin_39): track 0.00 -> 279.6 mm, vias 0 -> 2
- net Net-(J1-Pin_24): track 272.9 -> 0.00 mm, vias 2 -> 0
- net Net-(J1-Pin_6): track 261.9 -> 0.00 mm, vias 2 -> 0
- net Net-(J1-Pin_23): track 261.3 -> 0.00 mm, vias 1 -> 0
- net Net-(J1-Pin_4): track 253.8 -> 0.00 mm, vias 1 -> 0
- net Net-(J5-Pin_17): track 0.00 -> 253.2 mm, vias 0 -> 1
- net Net-(J1-Pin_22): track 248.2 -> 0.00 mm, vias 1 -> 0
- net Net-(J1-Pin_5): track 241.6 -> 0.00 mm, vias 3 -> 0
- net Net-(J5-Pin_19): track 0.00 -> 240.5 mm, vias 0 -> 1
- net Net-(J5-Pin_16): track 0.00 -> 236.4 mm, vias 0 -> 1
- net Net-(J5-Pin_18): track 0.00 -> 232.0 mm, vias 0 -> 2
- net Net-(J5-Pin_20): track 0.00 -> 228.6 mm, vias 0 -> 2
- net Net-(J5-Pin_34): track 0.00 -> 214.8 mm, vias 0 -> 1
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Other:
- board text added: "+12V Variable Backlight"
- board text added: "1"
- board text added: "40"
- board text added: "GND"
- board text added: "[CONNECTION J1] 1-RAT-MAN-ON-TOP_LED 2-RAT-MAN-ON-BOTTOM_LED 3-RAT-MAN-ON-KORRY_SW"
- board text added: "[CONNECTION J2] 1-ENG-1-PUMP-TOP_LED 2-ENG-1-PUMP-BOTTOM_LED 3-ENG-1-PUMP-KORRY_SW 4-L-TK-PUMPS-2-TOP_LED 5-L-TK-PUMPS-2-BOTTOM_LED 6-L-TK-PUMPS-2-KORRY_SW 7-ELEC-PUMP-TOP_LED 8-ELEC-PUMP-BOTTOM_LED 9-ELEC-PUMP-KORRY_SW 10-MODE_SEL-TOP_LED 11-MODE_SEL-BOTTOM_LED 12-MODE_SEL-KORRY_SW 13-CTR-TK-R-XFR-TOP_LED 14-CTR-TK-R-XFR-BOTTOM_LED 15-CTR-TK-R-XFR-KORRY_SW 16-R-RTK-PUMPS-1-TOP_LED 17-R-RTK-PUMPS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"
