File: overhead/centre/hyd-fuel/electronics/hyd-fuel.kicad_sch (KiCad schematic)
At the start: 144 parts, among them J1 Conn_02x20_Counter_Clockwise, J2 Conn_01x03_Pin, J3 Conn_02x01

Commit message: Changes
Changes
Parts:
- removed J1: Conn_02x20_Counter_Clockwise, Connector_PinHeader_2.54mm:PinHeader_2x20_P2.54mm_Vertical, symbol Connector_Generic:Conn_02x22_Counter_Clockwise
- removed J2: Conn_01x03_Pin, Connector_PinHeader_2.54mm:PinHeader_1x03_P2.54mm_Vertical, symbol Connector:Conn_01x03_Pin
- added J1, J5: Conn_02x20_Counter_Clockwise, Connector_PinHeader_2.54mm:PinHeader_2x20_P2.54mm_Vertical, symbol Connector_Generic:Conn_02x20_Counter_Clockwise
- added J4: Conn_02x01, TerminalBlock:TerminalBlock_bornier-2_P5.08mm, symbol Connector_Generic:Conn_02x01
- added KR14: ~, OpenA3XX:Korry Switch, symbol KorrySwitch:Korry_Switch
Connections:
- net +12V: now also J4.2 (Pin_2)
- net GND: now also J4.1 (Pin_1), KR14.2 (GND_TOP_LED), KR14.4 (GND_BOTTOM_LED), KR14.6 (SW_OUT)
- net at KR4.1 (+5V_TOP_LED): now also J5.25 (Pin_25)
- net at KR4.3 (+5V_BOTTOM_LED): now also J5.26 (Pin_26)
- net at KR4.5 (SW_IN): now also J5.27 (Pin_27)
- net at KR13.1 (+5V_TOP_LED): now also J5.19 (Pin_19)
- net at KR13.3 (+5V_BOTTOM_LED): now also J5.20 (Pin_20)
- net at KR13.5 (SW_IN): now also J5.21 (Pin_21)
- net at KR10.1 (+5V_TOP_LED): now also J5.34 (Pin_34)
- net at KR10.3 (+5V_BOTTOM_LED): now also J5.35 (Pin_35)
- net at KR10.5 (SW_IN): now also J5.36 (Pin_36)
- net at KR1.1 (+5V_TOP_LED): now also J5.1 (Pin_1)
- net at KR7.1 (+5V_TOP_LED): now also J5.10 (Pin_10)
- net at KR7.3 (+5V_BOTTOM_LED): now also J5.11 (Pin_11)
- net at KR7.5 (SW_IN): now also J5.12 (Pin_12)
- net at KR9.1 (+5V_TOP_LED): now also J5.13 (Pin_13)
- net at KR9.3 (+5V_BOTTOM_LED): now also J5.14 (Pin_14)
- net at KR9.5 (SW_IN): now also J5.15 (Pin_15)
- net at KR11.1 (+5V_TOP_LED): now also J5.16 (Pin_16)
- net at KR11.3 (+5V_BOTTOM_LED): now also J5.17 (Pin_17)
- net at KR11.5 (SW_IN): now also J5.18 (Pin_18)
- net at KR1.3 (+5V_BOTTOM_LED): now also J5.2 (Pin_2)
- net at KR2.1 (+5V_TOP_LED): now also J5.22 (Pin_22)
- net at KR2.3 (+5V_BOTTOM_LED): now also J5.23 (Pin_23)
- net at KR2.5 (SW_IN): now also J5.24 (Pin_24)
- net at KR6.1 (+5V_TOP_LED): now also J5.28 (Pin_28)
- net at KR6.3 (+5V_BOTTOM_LED): now also J5.29 (Pin_29)
- net at KR1.5 (SW_IN): now also J5.3 (Pin_3)
- net at KR6.5 (SW_IN): now also J5.30 (Pin_30)
- net at KR8.1 (+5V_TOP_LED): now also J5.31 (Pin_31)
- net at KR8.3 (+5V_BOTTOM_LED): now also J5.32 (Pin_32)
- net at KR8.5 (SW_IN): now also J5.33 (Pin_33)
- net at KR12.1 (+5V_TOP_LED): now also J5.37 (Pin_37)
- net at KR12.3 (+5V_BOTTOM_LED): now also J5.38 (Pin_38)
- net at KR12.5 (SW_IN): now also J5.39 (Pin_39)
- net at KR3.1 (+5V_TOP_LED): now also J5.4 (Pin_4)
- net at KR3.3 (+5V_BOTTOM_LED): now also J5.5 (Pin_5)
- net at KR3.5 (SW_IN): now also J5.6 (Pin_6)
- net at KR5.1 (+5V_TOP_LED): now also J5.7 (Pin_7)
- net at KR5.3 (+5V_BOTTOM_LED): now also J5.8 (Pin_8)
- net at KR5.5 (SW_IN): now also J5.9 (Pin_9)
- new net: J1.1 (Pin_1), KR14.1 (+5V_TOP_LED)
- new net: J1.2 (Pin_2), KR14.3 (+5V_BOTTOM_LED)
- new net: J1.3 (Pin_3), KR14.5 (SW_IN)
- no-connect marks 0 -> 38
Other:
- moved on the sheet: J3
