File: overhead/centre/fire/electronics/fire/fire.kicad_pcb (KiCad board)
At the start: 2 copper layers, 322.3 x 74.7 mm, 97 parts, among them J1 Conn_02x01, J2 Conn_02x20_Counter_Clockwise, J3 Conn_01x03_Pin, J4 Conn_01x03_Pin, J5 Conn_01x03_Pin, J6 Conn_01x03_Pin, J7 Conn_01x03_Pin, J8 Conn_01x03_Pin

Commit message: Fire PCB Updates - Iteration 2
Parts:
- added J9: Conn_02x01, TerminalBlock:TerminalBlock_bornier-2_P5.08mm, B.Cu at (77.5, 178.3)
Routing:
- net +12V: track 725.8 -> 695.9 mm, vias 12 -> 14
- net GND: track 800.9 -> 828.1 mm, vias 13 -> 11
- net Net-(J2-Pin_19): track 267.7 -> 247.6 mm
- net Net-(J2-Pin_2): track 312.2 -> 298.9 mm
- net Net-(J2-Pin_21): track 131.4 -> 144.1 mm
- net Net-(D19-K): track 30.5 -> 18.4 mm
- net Net-(D23-K): track 36.0 -> 46.1 mm
- net Net-(J2-Pin_7): track 189.6 -> 198.6 mm, vias 1 -> 4
- net Net-(J2-Pin_13): track 29.0 -> 37.8 mm, vias 0 -> 1
- net Net-(D30-K): track 58.9 -> 67.2 mm
- net Net-(D45-K): track 40.3 -> 48.3 mm
- net Net-(D44-K): track 26.7 -> 19.5 mm
- net Net-(D35-K): track 19.6 -> 12.9 mm, vias 2 -> 0
- net Net-(J2-Pin_4): track 198.5 -> 192.0 mm, vias 2 -> 1
- net Net-(J2-Pin_18): track 251.5 -> 258.0 mm
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Other:
- board text added: "+12V Variable Backlight"
- board text added: "1"
- board text added: "40"
- board text added: "GND"
- board text added: "[CONNECTION J2] 1-ENGINE-1-AGENT-1-TOP_LED 2-ENGINE-1-AGENT-1-BOTTOM_LED 3-ENGINE-1-AGENT-1-KORRY_SW 4-ENGINE-1-AGENT-2-TOP_LED 5-ENGINE-1-AGENT-2-BOTTOM_LED 6-ENGINE-1-AGENT-2-KORRY_SW 7-APU-AGENT-TOP_LED 8-APU-AGENT-BOTTOM_LED 9-APU-AGENT-KORRY_SW 10-ENGINE-2-AGENT-1-TOP_LED 11-ENGINE-2-AGENT-1-BOTTOM_LED 12-ENGINE-2-AGENT-1-KORRY_SW 13-ENGINE-2-AGENT-2-TOP_LED 14-ENGINE-2-AGENT-2-BOTTOM_LED 15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"
