File: overhead/centre/fire/electronics/fire/fire.kicad_sch (KiCad schematic)
At the start: 95 parts, among them J1 Conn_02x01, J2 Conn_02x20_Counter_Clockwise, J3 Conn_01x03_Pin, J4 Conn_01x03_Pin, J5 Conn_01x03_Pin, J6 Conn_01x03_Pin, J7 Conn_01x03_Pin, J8 Conn_01x03_Pin

Commit message: Fire PCB Updates - Iteration 2
Parts:
- added J9: Conn_02x01, TerminalBlock:TerminalBlock_bornier-2_P5.08mm, symbol Connector_Generic:Conn_02x01
Connections:
- net +12V: now also J9.2 (Pin_2)
- net GND: now also J9.1 (Pin_1)
- no-connect marks 0 -> 13
Changed lines of the file:
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@@
 		(color 0 0 0 0)
 	)
+	(junction
+		(at 50.8 187.96)
+		(diameter 0)
+		(color 0 0 0 0)
+	)
+	(no_connect
+		(at 134.62 31.75)
+	)
+	(no_connect
+		(at 134.62 36.83)
+	)
+	(no_connect
+		(at 134.62 46.99)
+	)
+	(no_connect
+		(at 134.62 54.61)
+	)
+	(no_connect
+		(at 134.62 41.91)
+	)
+	(no_connect
+		(at 134.62 49.53)
+	)
+	(no_connect
+		(at 134.62 59.69)
+	)
+	(no_connect
+		(at 134.62 34.29)
+	)
+	(no_connect
+		(at 134.62 57.15)
+	)
+	(no_connect
+		(at 134.62 29.21)
+	)
+	(no_connect
+		(at 134.62 44.45)
+	)
+	(no_connect
+		(at 134.62 52.07)
+	)
+	(no_connect
+		(at 134.62 39.37)
+	)
 	(wire
 		(pts
@@
 	(wire
 		(pts
+			(xy 38.1 187.96) (xy 50.8 187.96)
+		)
+		(stroke
+			(width 0)
+			(type default)
+		)
+	)
+	(wire
+		(pts
 			(xy 74.93 231.14) (xy 74.93 226.06)
 		)
@@
 	(wire
 		(pts
-			(xy 50.8 186.69) (xy 50.8 190.5)
+			(xy 50.8 186.69) (xy 50.8 187.96)
 		)
 		(stroke
@@
 	(wire
 		(pts
+			(xy 38.1 186.69) (xy 38.1 187.96)
+		)
+		(stroke
+			(width 0)
+			(type default)
+		)
+	)
+	(wire
+		(pts
 			(xy 148.59 350.52) (xy 148.59 353.06)
 		)
@@
 	(wire
 		(pts
+			(xy 38.1 172.72) (xy 50.8 172.72)
+		)
+		(stroke
+			(width 0)
+			(type default)
+		)
+	)
+	(wire
+		(pts
 			(xy 104.14 274.32) (xy 104.14 269.24)
 		)
@@
 	(wire
 		(pts
+			(xy 50.8 187.96) (xy 50.8 190.5)
+		)
+		(stroke
+			(width 0)
+			(type default)
+		)
+	)
+	(wire
+		(pts
 			(xy 175.26 128.27) (xy 157.48 128.27)
 		)
@@
 	(wire
 		(pts
+			(xy 38.1 173.99) (xy 38.1 172.72)
+		)
+		(stroke
+			(width 0)
+			(type default)
+		)
+	)
+	(wire
+		(pts
 			(xy 62.23 316.23) (xy 52.07 316.23)
 		)
@@
 	)
 	(symbol
+		(lib_id "Connector_Generic:Conn_02x01")
+		(at 38.1 181.61 90)
+		(unit 1)
+		(exclude_from_sim no)
+		(in_bom yes)
+		(on_board yes)
+		(dnp no)
+		(property "Reference" "J9"
+			(at 32.5882 180.34 0)
+			(effects
+				(font
+					(size 1.27 1.27)
+				)
+			)
+		)
+		(property "Value" "Conn_02x01"
+			(at 34.8996 180.34 0)
+			(effects
+				(font
+					(size 1.27 1.27)
+				)
+			)
+		)
+		(property "Footprint" "TerminalBlock:TerminalBlock_bornier-2_P5.08mm"
+			(at 38.1 181.61 0)
+			(effects
+				(font
+					(size 1.27 1.27)
+				)
+				(hide yes)
+			)
+		)
+		(property "Datasheet" "~"
+			(at 38.1 181.61 0)
+			(effects
+				(font
+					(size 1.27 1.27)
+				)
+				(hide yes)
+			)
+		)
+		(property "Description" "Generic connector, double row, 02x01, this symbol is compatible with counter-clockwise, top-bottom and odd-even numbering schemes., script generated (kicad-library-utils/schlib/autogen/connector/)"
+			(at -17.78 175.26 0)
+			(effects
+				(font
+					(size 1.27 1.27)
+				)
+				(hide yes)
+			)
+		)
+		(pin "1"
+		)
+		(pin "2"
+		)
+		(instances
+			(project "fire"
+				(path "/3f476c7a-4a20-4caf-b3a4-c9516a17c804"
+					(reference "J9")
+					(unit 1)
+				)
+			)
+		)
+	)
+	(symbol
 		(lib_id "power:+12V")
 		(at 213.36 300.99 0)
@@
 		(on_board yes)
 		(dnp no)
-		(fields_autoplaced yes)
 		(property "Reference" "J5"
 			(at 230.505 64.77 0)
@@
 			)
 		)
-		(property "Description" "Strobe"
-			(at 231.14 57.15 0)
+		(property "Description" "APU Fire"
+			(at 236.22 57.15 0)
 			(effects
 				(font
@@
 		(on_board yes)
 		(dnp no)
-		(fields_autoplaced yes)
 		(property "Reference" "J4"
 			(at 230.505 49.53 0)
@@
 			)
 		)
-		(property "Description" "Strobe"
-			(at 231.14 41.91 0)
+		(property "Description" "Engine 1 Fire"
+			(at 238.76 41.91 0)
 			(effects
 				(font
@@
 		(on_board yes)
 		(dnp no)
-		(fields_autoplaced yes)
 		(property "Reference" "J3"
 			(at 230.505 33.02 0)
@@
 			)
 		)
-		(property "Description" "Strobe"
-			(at 231.14 25.4 0)
+		(property "Description" "Engine 1 Test"
+			(at 239.014 25.4 0)
 			(effects
 				(font
@@
 		(on_board yes)
 		(dnp no)
-		(fields_autoplaced yes)
 		(property "Reference" "J7"
 			(at 230.505 97.79 0)
@@
 			)
 		)
-		(property "Description" "Strobe"
-			(at 231.14 90.17 0)
+		(property "Description" "Engine 2 Fire"
+			(at 238.252 90.424 0)
 			(effects
 				(font
@@
 		(on_board yes)
 		(dnp no)
-		(fields_autoplaced yes)
 		(property "Reference" "J6"
 			(at 230.505 81.28 0)
@@
 			)
 		)
-		(property "Description" "Strobe"
-			(at 231.14 73.66 0)
+		(property "Description" "APU Test"
+			(at 236.22 73.66 0)
 			(effects
 				(font
@@
 		(on_board yes)
 		(dnp no)
-		(fields_autoplaced yes)
 		(property "Reference" "KR5"
 			(at 246.38 135.2549 0)
@@
 			)
 		)
-		(property "Description" "Cabin Press Mode Sel"
-			(at 234.95 127 0)
+		(property "Description" "Engine 2 Agent 2"
+			(at 236.22 126.492 0)
 			(effects
 				(font
@@
 		(on_board yes)
 		(dnp no)
-		(fields_autoplaced yes)
 		(property "Reference" "KR4"
-			(at 196.85 133.9849 0)
+			(at 196.85 132.7149 0)
 			(effects
 				(font
@@
 		)
 		(property "Value" "~"
-			(at 196.85 135.89 0)
+			(at 196.85 134.62 0)
 			(effects
 				(font
@@
 			)
 		)
-		(property "Description" "Probe Window Heat"
-			(at 185.42 125.73 0)
+		(property "Description" "Engine 2 Agent 1"
+			(at 178.308 125.222 0)
 			(effects
 				(font
 					(size 1.27 1.27)
 				)
+				(justify left)
 			)
 		)
@@
 		(on_board yes)
 		(dnp no)
-		(fields_autoplaced yes)
 		(property "Reference" "KR2"
-			(at 109.22 133.9849 0)
+			(at 109.22 132.7149 0)
 			(effects
 				(font
@@
 		)
 		(property "Value" "~"
-			(at 109.22 135.89 0)
+			(at 109.22 134.62 0)
 			(effects
 				(font
@@
 			)
 		)
-		(property "Description" "Anti-Ice Eng 1"
-			(at 97.79 125.73 0)
+		(property "Description" "Engine 1 Agent 2"
+			(at 90.424 125.222 0)
 			(effects
 				(font
 					(size 1.27 1.27)
 				)
+				(justify left)
 			)
 		)
@@
 		(on_board yes)
 		(dnp no)
-		(fields_autoplaced yes)
 		(property "Reference" "J8"
 			(at 230.505 114.3 0)
@@
 			)
 		)
-		(property "Description" "Strobe"
-			(at 231.14 106.68 0)
+		(property "Description" "Engine 2 Test"
+			(at 238.506 106.934 0)
 			(effects
 				(font
@@
 			)
 		)
-		(property "Description" "Anti-Ice Wing"
-			(at 50.038 124.968 0)
+		(property "Description" "Engine 1 Agent 1"
+			(at 48.006 125.222 0)
 			(effects
 				(font
@@
 		(on_board yes)
 		(dnp no)
-		(fields_autoplaced yes)
 		(property "Reference" "KR3"
-			(at 156.21 133.9849 0)
+			(at 156.21 132.7149 0)
 			(effects
 				(font
@@
 		)
 		(property "Value" "~"
-			(at 156.21 135.89 0)
+			(at 156.21 134.62 0)
 			(effects
 				(font
@@
 			)
 		)
-		(property "Description" "Anti-Ice Eng 2"
-			(at 144.78 125.73 0)
+		(property "Description" "APU Agent"
+			(at 140.716 125.476 0)
 			(effects
 				(font
 					(size 1.27 1.27)
 				)
+				(justify left)
 			)
 		)
