File: overhead/right/flt-ctl-fo/electronics/flt-ctl-fo.kicad_pcb (KiCad board)
At the start: 2 copper layers, 145 x 47.3 mm, 48 parts, among them J1 Conn_02x01, J2 Conn_02x20_Counter_Clockwise

Commit message: FLT-CTL FO Side Iteration 2
Parts:
- added J3: Conn_02x01, TerminalBlock:TerminalBlock_bornier-2_P5.08mm, B.Cu at (84.5, 119.6)
- moved LogoBottom 134.0 mm to (213.9, 101.3), turned to 90 degrees
- moved LogoTop 134.0 mm to (213.9, 101.3), turned to -90 degrees
Routing:
- net +12V: track 296.2 -> 330.6 mm, vias 4 -> 8
- net Net-(D17-K): track 36.6 -> 11.4 mm, vias 0 -> 2
- net Net-(J2-Pin_9): track 82.3 -> 66.4 mm, vias 2 -> 1
- net Net-(D16-K): track 61.7 -> 76.7 mm
- net Net-(D2-K): track 22.1 -> 11.8 mm, vias 2 -> 0
- net Net-(D20-K): track 34.9 -> 43.6 mm
- net Net-(D9-K): track 6.37 -> 14.8 mm, vias 0 -> 2
- net Net-(J2-Pin_2): track 135.4 -> 128.1 mm
- net Net-(D8-K): track 23.1 -> 17.9 mm
- net Net-(D30-K): track 23.3 -> 27.3 mm
- net Net-(D12-K): track 18.2 -> 14.3 mm
- net Net-(D26-K): track 19.8 -> 16.1 mm
- net Net-(D23-K): track 18.6 -> 15.1 mm, vias 2 -> 0
- net Net-(J2-Pin_6): track 111.5 -> 108.2 mm
- net Net-(J2-Pin_8): track 56.3 -> 58.9 mm
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Other:
- board text added: "+12V Variable Backlight"
- board text added: "1"
- board text added: "40"
- board text added: "GND"
- board text added: "[CONNECTION J2] 1-ELAC2-TOP_LED 2-ELAC2-BOTTOM_LED 3-ELAC2-KORRY_SW 4-SEC2-TOP_LED 5-SEC2-BOTTOM_LED 6-SEC2-KORRY_SW 7-SEC3-TOP_LED 8-SEC3-BOTTOM_LED 9-SEC3-KORRY_SW 10-FAC2-TOP_LED 11-FAC2-BOTTOM_LED 12-FAC2-KORRY_SW"
