File: overhead/right/flt-ctl-fo/electronics/flt-ctl-fo.kicad_sch (KiCad schematic)
At the start: 46 parts, among them J1 Conn_02x01, J2 Conn_02x20_Counter_Clockwise

Commit message: FLT-CTL FO Side Iteration 2
Parts:
- added J3: Conn_02x01, TerminalBlock:TerminalBlock_bornier-2_P5.08mm, symbol Connector_Generic:Conn_02x01
Connections:
- net +12V: now also J3.2 (Pin_2)
- net GND: now also J3.1 (Pin_1)
- no-connect marks 1 -> 28
Changed lines of the file:
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@@
 	)
 	(junction
+		(at 85.09 80.01)
+		(diameter 0)
+		(color 0 0 0 0)
+	)
+	(junction
 		(at 167.64 181.61)
 		(diameter 0)
@@
 	)
 	(no_connect
+		(at 142.24 111.76)
+	)
+	(no_connect
+		(at 142.24 132.08)
+	)
+	(no_connect
+		(at 142.24 137.16)
+	)
+	(no_connect
+		(at 142.24 152.4)
+	)
+	(no_connect
+		(at 142.24 154.94)
+	)
+	(no_connect
+		(at 142.24 124.46)
+	)
+	(no_connect
+		(at 142.24 119.38)
+	)
+	(no_connect
+		(at 129.54 149.86)
+	)
+	(no_connect
+		(at 142.24 134.62)
+	)
+	(no_connect
 		(at 142.24 106.68)
 	)
+	(no_connect
+		(at 142.24 129.54)
+	)
+	(no_connect
+		(at 129.54 152.4)
+	)
+	(no_connect
+		(at 129.54 137.16)
+	)
+	(no_connect
+		(at 142.24 109.22)
+	)
+	(no_connect
+		(at 129.54 147.32)
+	)
+	(no_connect
+		(at 142.24 149.86)
+	)
+	(no_connect
+		(at 142.24 142.24)
+	)
+	(no_connect
+		(at 129.54 144.78)
+	)
+	(no_connect
+		(at 129.54 154.94)
+	)
+	(no_connect
+		(at 142.24 121.92)
+	)
+	(no_connect
+		(at 142.24 144.78)
+	)
+	(no_connect
+		(at 142.24 139.7)
+	)
+	(no_connect
+		(at 129.54 142.24)
+	)
+	(no_connect
+		(at 129.54 139.7)
+	)
+	(no_connect
+		(at 142.24 127)
+	)
+	(no_connect
+		(at 142.24 147.32)
+	)
+	(no_connect
+		(at 142.24 114.3)
+	)
+	(no_connect
+		(at 142.24 116.84)
+	)
 	(wire
 		(pts
@@
 	(wire
 		(pts
+			(xy 85.09 80.01) (xy 85.09 82.55)
+		)
+		(stroke
+			(width 0)
+			(type default)
+		)
+	)
+	(wire
+		(pts
+			(xy 74.93 64.77) (xy 85.09 64.77)
+		)
+		(stroke
+			(width 0)
+			(type default)
+		)
+	)
+	(wire
+		(pts
 			(xy 73.66 267.97) (xy 96.52 267.97)
 		)
@@
 	(wire
 		(pts
+			(xy 74.93 66.04) (xy 74.93 64.77)
+		)
+		(stroke
+			(width 0)
+			(type default)
+		)
+	)
+	(wire
+		(pts
 			(xy 118.11 273.05) (xy 118.11 275.59)
 		)
@@
 	(wire
 		(pts
+			(xy 74.93 80.01) (xy 85.09 80.01)
+		)
+		(stroke
+			(width 0)
+			(type default)
+		)
+	)
+	(wire
+		(pts
 			(xy 297.18 252.73) (xy 307.34 252.73)
 		)
@@
 	(wire
 		(pts
-			(xy 85.09 78.74) (xy 85.09 82.55)
+			(xy 85.09 78.74) (xy 85.09 80.01)
 		)
 		(stroke
@@
 	(wire
 		(pts
+			(xy 74.93 78.74) (xy 74.93 80.01)
+		)
+		(stroke
+			(width 0)
+			(type default)
+		)
+	)
+	(wire
+		(pts
 			(xy 162.56 273.05) (xy 170.18 273.05)
 		)
@@
 					(unit 1)
 				)
+			)
+		)
+	)
+	(symbol
+		(lib_id "Connector_Generic:Conn_02x01")
+		(at 74.93 73.66 90)
+		(unit 1)
+		(exclude_from_sim no)
+		(in_bom yes)
+		(on_board yes)
+		(dnp no)
+		(property "Reference" "J3"
+			(at 69.4182 72.39 0)
+			(effects
+				(font
+					(size 1.27 1.27)
+				)
+			)
+		)
+		(property "Value" "Conn_02x01"
+			(at 71.7296 72.39 0)
+			(effects
+				(font
+					(size 1.27 1.27)
+				)
+			)
+		)
+		(property "Footprint" "TerminalBlock:TerminalBlock_bornier-2_P5.08mm"
+			(at 74.93 73.66 0)
+			(effects
+				(font
+					(size 1.27 1.27)
+				)
+				(hide yes)
+			)
+		)
+		(property "Datasheet" "~"
+			(at 74.93 73.66 0)
+			(effects
+				(font
+					(size 1.27 1.27)
+				)
+				(hide yes)
+			)
+		)
+		(property "Description" "Generic connector, double row, 02x01, this symbol is compatible with counter-clockwise, top-bottom and odd-even numbering schemes., script generated (kicad-library-utils/schlib/autogen/connector/)"
+			(at 19.05 67.31 0)
+			(effects
+				(font
+					(size 1.27 1.27)
+				)
+				(hide yes)
+			)
+		)
+		(pin "1"
+		)
+		(pin "2"
+		)
+		(instances
+			(project "flt-ctl-fo"
+				(path "/6e16cde8-5baf-476b-b1e1-4399c233ed4c"
+					(reference "J3")
+					(unit 1)
+				)
