File: overhead/right/cargo-vent_cargo-smoke/electronics/cargo-vent_cargo-smoke.kicad_pcb (KiCad board)
At the start: 2 copper layers, 145 x 127.5 mm, 66 parts, among them J1 Conn_02x01, J2 Conn_02x20_Counter_Clockwise, J3 Conn_02x01, J4 Conn_02x01, J5 Conn_02x01

Commit message: Cargo Vent and Cargo Smoke Panel Iteration 2
Parts:
- removed J5: Conn_02x01, Connector_PinHeader_2.54mm:PinHeader_1x02_P2.54mm_Vertical
- added KR4: ~, OpenA3XX:Korry Switch, F.Cu at (151.1, 200.6)
- added KR5: ~, OpenA3XX:Korry Switch, F.Cu at (250.3, 200.6)
- J3: footprint Connector_PinHeader_2.54mm:PinHeader_1x02_P2.54mm_Vertical -> TerminalBlock:TerminalBlock_bornier-2_P5.08mm; moved to B.Cu
- moved J3 21.8 mm to (166.9, 226.5), turned to 180 degrees
Connections:
- J3 pad 2: Net-(J2-Pin_10) -> +12V
Routing:
- net +12V: track 530.4 -> 513.5 mm, vias 8 -> 9
- net Net-(D16-K): track 31.5 -> 42.8 mm, vias 0 -> 2
- net Net-(J2-Pin_1): track 165.9 -> 174.7 mm, vias 2 -> 1
- net Net-(D21-K): track 25.1 -> 32.6 mm, vias 0 -> 2
- net Net-(J2-Pin_2): track 159.7 -> 167.0 mm
- net Net-(D36-K): track 18.2 -> 11.5 mm, vias 2 -> 0
- net Net-(D35-K): track 14.8 -> 8.39 mm
- net Net-(J2-Pin_11): track 117.7 -> 123.3 mm
- net Net-(J2-Pin_6): track 66.8 -> 72.1 mm
- net Net-(J2-Pin_12): track 161.5 -> 156.3 mm
- net Net-(D39-K): track 19.5 -> 24.7 mm, vias 0 -> 2
- net Net-(J2-Pin_4): track 82.1 -> 77.4 mm
- net Net-(D19-K): track 26.1 -> 21.8 mm, vias 2 -> 0
- net Net-(D22-K): track 34.5 -> 38.7 mm
- net Net-(J2-Pin_9): track 126.7 -> 122.9 mm
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Other:
- board text added: "+12V Variable Backlight"
- board text added: "1"
- board text added: "40"
- board text added: "GND"
- board text added: "[CONNECTION J2] 1-AFT-ISOL-VALVE-TOP_LED 2-AFT-ISOL-VALVE-BOTTOM_LED 3-AFT-ISOL-VALVE-KORRY_SW 4-CARGO-SMOKE-FWD-1-TOP_LED 5-CARGO-SMOKE-FWD-1-BOTTOM_LED 6-CARGO-SMOKE-FWD-1-KORRY_SW 7-CARGO-SMOKE-FWD-2-TOP_LED 8-CARGO-SMOKE-FWD-2-BOTTOM_LED 9-CARGO-SMOKE-FWD-2-KORRY_SW 10-CARGO-SMOKE-DISCHARGE-1-KORRY_SW 11-CARGO-SMOKE-TEST_SW 12-CARGO-SMOKE-DISCHARGE-2-KORRY_SW"
