File: overhead/right/cargo-vent_cargo-smoke/electronics/cargo-vent_cargo-smoke.kicad_sch (KiCad schematic)
At the start: 64 parts, among them J1 Conn_02x01, J2 Conn_02x20_Counter_Clockwise, J3 Conn_02x01, J4 Conn_02x01, J5 Conn_02x01

Commit message: Cargo Vent and Cargo Smoke Panel Iteration 2
Parts:
- removed J5: Conn_02x01, Connector_PinHeader_2.54mm:PinHeader_1x02_P2.54mm_Vertical, symbol Connector_Generic:Conn_02x01
- added KR4, KR5: ~, OpenA3XX:Korry Switch, symbol KorrySwitch:Korry_Switch
- J3: footprint Connector_PinHeader_2.54mm:PinHeader_1x02_P2.54mm_Vertical -> TerminalBlock:TerminalBlock_bornier-2_P5.08mm
Connections:
- net +12V: now also J3.2 (Pin_2)
- net GND: now also KR4.6 (SW_OUT), KR5.6 (SW_OUT)
- net at J2.10 (Pin_10): now also KR4.5 (SW_IN); no longer J3.2 (Pin_2)
- net at J2.12 (Pin_12): now also KR5.5 (SW_IN)
- no-connect marks 0 -> 36
Other:
- note added: "AFT ISOL VALVE"
- note added: "CARGO SMOKE DISCHARGE 1"
- note added: "CARGO SMOKE DISCHARGE 2"
- note added: "CARGO SMOKE FWD 1"
- note added: "CARGO SMOKE FWD 2"
- note added: "CARGO SMOKE TEST"
