File: overhead/right/ventilation_eng_rain-rplnt_wipers/electronics/a320-overhead-ventilation_eng_rain-rplnt-wipers.kicad_sch (KiCad schematic)
At the start: 69 parts, among them J1 Conn_02x01, J2 Conn_02x20_Counter_Clockwise, J3 Conn_02x01, J4 Conn_02x02_Counter_Clockwise

Commit message: Updates
Parts:
- added J5: Conn_02x01, TerminalBlock:TerminalBlock_bornier-2_P5.08mm, symbol Connector_Generic:Conn_02x01
Connections:
- net +12V: now also J5.2 (Pin_2)
- net GND: now also J5.1 (Pin_1)
- no-connect marks 0 -> 22
Other:
- note added: "Blower"
- note added: "Cab Fans"
- note added: "Extract"
- note added: "Man Start 1"
- note added: "Man Start 2"
- note added: "Rain Rplnt"
- note added: "Wiper"
